File: Hardware/12VBoard_2021_Rev1/High Current Outputs.sch (KiCad schematic (older format))
At the start: 0 parts

Commit message: BD9811MUV symbol made along with most supporting circuits
Parts:
- added C? (x2): 10uF, symbol pspice:CAP
- added C? (x3): 0.1uF, symbol pspice:CAP
- added U?: BD9611MUV, symbol Converter_DCDC:BD9611MUV
Connections:
- net labels added: +12V
Changed lines of the file:
@@
 $Descr A4 11693 8268
 encoding utf-8
-Sheet 1 3
+Sheet 3 4
 Title ""
 Date ""
@@
 Comment4 ""
 $EndDescr
+$Comp
+L Converter_DCDC:BD9611MUV U?
+U 1 1 5F7A443F
+P 2800 2300
+F 0 "U?" H 2800 2400 50  0000 C CNN
+F 1 "BD9611MUV" H 2800 2300 50  0000 C CNN
+F 2 "" H 2800 2450 50  0001 C CNN
+F 3 "" H 2800 2450 50  0001 C CNN
+	1    2800 2300
+	1    0    0    -1
+$EndComp
+$Comp
+L power:+12V #PWR?
+U 1 1 5F7A8A51
+P 4950 1250
+F 0 "#PWR?" H 4950 1100 50  0001 C CNN
+F 1 "+12V" H 4965 1423 50  0000 C CNN
+F 2 "" H 4950 1250 50  0001 C CNN
+F 3 "" H 4950 1250 50  0001 C CNN
+	1    4950 1250
+	1    0    0    -1
+$EndComp
+$Comp
+L pspice:CAP C?
+U 1 1 5F7ABCCA
+P 4500 1400
+F 0 "C?" H 4678 1446 50  0000 L CNN
+F 1 "10uF" H 4678 1355 50  0000 L CNN
+F 2 "" H 4500 1400 50  0001 C CNN
+F 3 "~" H 4500 1400 50  0001 C CNN
+	1    4500 1400
+	1    0    0    -1
+$EndComp
+$Comp
+L pspice:CAP C?
+U 1 1 5F7AD602
+P 4150 1400
+F 0 "C?" H 4328 1446 50  0000 L CNN
+F 1 "10uF" H 4328 1355 50  0000 L CNN
+F 2 "" H 4150 1400 50  0001 C CNN
+F 3 "~" H 4150 1400 50  0001 C CNN
+	1    4150 1400
+	1    0    0    -1
+$EndComp
+$Comp
+L pspice:CAP C?
+U 1 1 5F7B3804
+P 1650 2200
+F 0 "C?" V 1965 2200 50  0000 C CNN
+F 1 "0.1uF" V 1874 2200 50  0000 C CNN
+F 2 "" H 1650 2200 50  0001 C CNN
+F 3 "~" H 1650 2200 50  0001 C CNN
+	1    1650 2200
+	0    -1   -1   0
+$EndComp
+$Comp
+L pspice:CAP C?
+U 1 1 5F7B40C6
+P 1650 2600
+F 0 "C?" V 1965 2600 50  0000 C CNN
+F 1 "0.1uF" V 1874 2600 50  0000 C CNN
+F 2 "" H 1650 2600 50  0001 C CNN
+F 3 "~" H 1650 2600 50  0001 C CNN
+	1    1650 2600
+	0    -1   -1   0
+$EndComp
+$Comp
+L pspice:CAP C?
+U 1 1 5F7B4505
+P 1650 3000
+F 0 "C?" V 1965 3000 50  0000 C CNN
+F 1 "0.1uF" V 1874 3000 50  0000 C CNN
+F 2 "" H 1650 3000 50  0001 C CNN
+F 3 "~" H 1650 3000 50  0001 C CNN
+	1    1650 3000
+	0    -1   -1   0
+$EndComp
 $EndSCHEMATC
