File: Hardware/12VBoard_2021_Rev1/High Current Outputs.sch (KiCad schematic (older format))
At the start: 4 parts

Commit message: packVoltage line not connected in schematic
Sheet pins were used instead of hierarchical pins, which caused the line to not be continuous. Now it is connected
Changed lines of the file:
@@
 EESchema Schematic File Version 4
+LIBS:12VBoard_2021_Rev1-cache
 EELAYER 30 0
 EELAYER END
@@
 Text HLabel 3250 5275 0    79   Input ~ 16
 PackVoltage
-Text HLabel 5100 4875 2    50   Input ~ 0
-PackVoltage
-Text HLabel 6600 4875 2    50   Input ~ 0
-PackVoltage
 Wire Wire Line
 	6500 5275 6500 4875
@@
 Wire Wire Line
 	5000 5275 6500 5275
-$Sheet
-S 6600 3525 1250 1450
-U 5F8236F9
-F0 "Multimedia/Extra" 50
-F1 "MultimediaExtra.sch" 50
-F2 "12V10AMultimedia" O R 7850 3675 50
-F3 "CTL_MultimediaExtra" O R 7850 3825 50
-F4 "12V10AExtra" O R 7850 3750 50
-F5 "MultimediaExtraSense" O R 7850 3900 50
-F6 "5V" O L 6600 4775 49
-F7 "12V3AMultimediaExtraLogic" O R 7850 3600 50
-$EndSheet
 $Comp
 L MRDT_Connectors:AndersonPP Conn?
@@
 Wire Wire Line
 	3250 5275 3450 5275
-$Sheet
-S 3550 3525 1100 1450
-U 5F971CD6
-F0 "Gimbal" 50
-F1 "Gimbal.sch" 50
-F2 "CTL_Gimbal" I R 4650 3750 49
-F3 "12V5AGimbal" O R 4650 3675 49
-F4 "PackVoltage" I L 3550 4875 49
-F5 "GimbalSense" O R 4650 3825 49
-F6 "12V3AGimbalLogic" O R 4650 3600 50
-F7 "5V" I L 3550 4800 50
-$EndSheet
 Text HLabel 4875 3925 3    50   Input ~ 0
 GimbalCTL
@@
 Wire Wire Line
 	7950 3900 7850 3900
+Wire Wire Line
+	3250 5475 3400 5475
+Wire Wire Line
+	3550 4800 3400 4800
+Wire Wire Line
+	3400 4800 3400 5475
+Connection ~ 3400 5475
+Wire Wire Line
+	3400 5475 4950 5475
 $Sheet
 S 5100 3525 1250 1450
@@
 F3 "CTL_AuxMount" O R 6350 3750 50
 F4 "AuxMountSense" O R 6350 3825 50
-F5 "5V" O L 5100 4775 49
+F5 "5V" I L 5100 4775 49
 F6 "12V3AAuxMountLogic" O R 6350 3600 50
+F7 "PackVoltage" I L 5100 4875 50
 $EndSheet
-Wire Wire Line
-	3250 5475 3400 5475
-Wire Wire Line
-	3550 4800 3400 4800
-Wire Wire Line
-	3400 4800 3400 5475
-Connection ~ 3400 5475
-Wire Wire Line
-	3400 5475 4950 5475
+$Sheet
+S 3550 3525 1100 1450
+U 5F971CD6
+F0 "Gimbal" 50
+F1 "Gimbal.sch" 50
+F2 "CTL_Gimbal" I R 4650 3750 49
+F3 "12V5AGimbal" O R 4650 3675 49
+F4 "GimbalSense" O R 4650 3825 49
+F5 "12V3AGimbalLogic" O R 4650 3600 50
+F6 "5V" I L 3550 4800 50
+F7 "PackVoltage" I L 3550 4875 50
+$EndSheet
+$Sheet
+S 6600 3525 1250 1450
+U 5F8236F9
+F0 "Multimedia/Extra" 50
+F1 "MultimediaExtra.sch" 50
+F2 "12V10AMultimedia" O R 7850 3675 50
+F3 "CTL_MultimediaExtra" O R 7850 3825 50
+F4 "12V10AExtra" O R 7850 3750 50
+F5 "MultimediaExtraSense" O R 7850 3900 50
+F6 "5V" I L 6600 4775 49
+F7 "12V3AMultimediaExtraLogic" O R 7850 3600 50
+F8 "PackVoltage" I L 6600 4875 50
+$EndSheet
 $EndSCHEMATC
