File: Hardware/12VBoard_2021_Rev1/BBB&Switch.sch (KiCad schematic (older format))
At the start: 5 parts, among them U3 LM2576D2TR4

Commit message: YELLED AT DAN WITHOUT HIM HERE
Parts:
- U3: symbol MRDT_Devices:LM2576D2TR4 -> 12VBoard_2021_Rev1-rescue:LM2576D2TR4-MRDT_Devices
Changed lines of the file:
@@
 $Descr A4 11693 8268
 encoding utf-8
-Sheet 7 13
+Sheet 10 13
 Title ""
 Date ""
@@
 $EndComp
 $Comp
-L MRDT_Devices:LM2576D2TR4 U?
+L 12VBoard_2021_Rev1-rescue:LM2576D2TR4-MRDT_Devices U?
 U 1 1 5F7FBB26
 P 4950 3500
@@
 AR Path="/5F74F223/5F7E1E8A/5F7FBB26" Ref="U?"  Part="1"
 AR Path="/5F74F223/5F7D1499/5F7FBB26" Ref="U3"  Part="1"
+AR Path="/5F7FBB26" Ref="U3"  Part="1"
 F 0 "U3" H 4950 3925 50  0000 C CNN
 F 1 "LM2576D2TR4" H 4950 3834 50  0000 C CNN
