File: Hardware/12VBoard_2021_Rev1/Cam1&2.sch (KiCad schematic (older format))
At the start: 5 parts, among them U5 LM2576D2TR4

Commit message: YELLED AT DAN WITHOUT HIM HERE
Parts:
- U5: symbol MRDT_Devices:LM2576D2TR4 -> 12VBoard_2021_Rev1-rescue:LM2576D2TR4-MRDT_Devices
Changed lines of the file:
@@
 $EndComp
 $Comp
-L MRDT_Devices:LM2576D2TR4 U5
+L 12VBoard_2021_Rev1-rescue:LM2576D2TR4-MRDT_Devices U5
 U 1 1 5F7D90ED
 P 4500 2900
 AR Path="/5F74F223/5F7D1238/5F7D90ED" Ref="U5"  Part="1"
 AR Path="/5F74F223/5F7E1E8A/5F7D90ED" Ref="U?"  Part="1"
+AR Path="/5F7D90ED" Ref="U5"  Part="1"
 F 0 "U5" H 4500 3325 50  0000 C CNN
 F 1 "LM2576D2TR4" H 4500 3234 50  0000 C CNN
