File: Hardware/12VBoard_2021_Rev1/Extra.sch (KiCad schematic (older format))
At the start: 6 parts, among them SW1 SW_SPDT, U4 LM2576D2TR4

Commit message: YELLED AT DAN WITHOUT HIM HERE
Parts:
- U4: symbol MRDT_Devices:LM2576D2TR4 -> 12VBoard_2021_Rev1-rescue:LM2576D2TR4-MRDT_Devices
Connections:
- wire segments 36 -> 39
Other:
- moved on the sheet: C21, C22, D3, L4, SW1
