File: Hardware/12VBoard_2021_Rev1/Nav.sch (KiCad schematic (older format))
At the start: 5 parts, among them U2 LM2576D2TR4

Commit message: YELLED AT DAN WITHOUT HIM HERE
Parts:
- U2: symbol MRDT_Devices:LM2576D2TR4 -> 12VBoard_2021_Rev1-rescue:LM2576D2TR4-MRDT_Devices
Changed lines of the file:
@@
 $EndComp
 $Comp
-L MRDT_Devices:LM2576D2TR4 U?
+L 12VBoard_2021_Rev1-rescue:LM2576D2TR4-MRDT_Devices U?
 U 1 1 5F7FC664
 P 5250 3850
@@
 AR Path="/5F74F223/5F7E1E8A/5F7FC664" Ref="U?"  Part="1"
 AR Path="/5F74F223/5F7D1463/5F7FC664" Ref="U2"  Part="1"
+AR Path="/5F7FC664" Ref="U2"  Part="1"
 F 0 "U2" H 5250 4275 50  0000 C CNN
 F 1 "LM2576D2TR4" H 5250 4184 50  0000 C CNN
