File: Hardware/12VBoard_2021_Rev1/Tiva.sch (KiCad schematic (older format))
At the start: 0 parts

Commit message: current sense
started current sense circuit on hig current. added fuse and LED signal. started tiva wiring.
Parts:
- added Conn?: Molex_SL_10, symbol MRDT_Connectors:Molex_SL_10
Other:
- note added: "Tiva 4 analog(current sense)/ \n5 toggles(digital write)"
Changed lines of the file:
@@
 Comment4 ""
 $EndDescr
+$Comp
+L MRDT_Connectors:Molex_SL_10 Conn?
+U 1 1 5F9BCEA4
+P 4250 3100
+F 0 "Conn?" H 4378 3658 60  0000 L CNN
+F 1 "Molex_SL_10" H 4378 3552 60  0000 L CNN
+F 2 "" H 4250 3600 60  0001 C CNN
+F 3 "" H 4250 3600 60  0001 C CNN
+	1    4250 3100
+	1    0    0    -1
+$EndComp
+Text Notes 4400 2950 0    79   ~ 0
+Tiva 4 analog(current sense)/ \n5 toggles(digital write)
 $EndSCHEMATC
