File: Hardware/12VBoard_2021_Rev1/Tiva.sch (KiCad schematic (older format))
At the start: 2 parts

Commit message: admin changes
-current sensing on high current
-fixed traces for current sensing
Parts:
- removed Conn2: Molex_SL_04, MRDT_Connectors:MOLEX_SL_04_Horizontal, symbol MRDT_Connectors:Molex_SL_04
- added Conn?: Molex_SL_05, symbol MRDT_Connectors:Molex_SL_05
Connections:
- net AuxMountSense: now also Conn?.2
- net GimbalSense: now also Conn?.3
- net LowCurrentSense: now also Conn?.4
- net MultimediaSense: now also Conn?.1
- new net CurrentSenseHigh: Conn?.5
Changed lines of the file:
@@
 EESchema Schematic File Version 4
+LIBS:12VBoard_2021_Rev1-cache
 EELAYER 30 0
 EELAYER END
 $Descr A4 11693 8268
 encoding utf-8
-Sheet 9 8
+Sheet 7 8
 Title ""
 Date ""
@@
 F 3 "" H 6450 5200 60  0001 C CNN
 	1    6450 4700
-	1    0    0    -1
-$EndComp
-$Comp
-L MRDT_Connectors:Molex_SL_04 Conn2
-U 1 1 5FB5B79F
-P 6450 5350
-F 0 "Conn2" H 6350 5175 60  0000 L CNN
-F 1 "Molex_SL_04" H 6175 5275 60  0000 L CNN
-F 2 "MRDT_Connectors:MOLEX_SL_04_Horizontal" H 6450 5350 60  0001 C CNN
-F 3 "" H 6450 5350 60  0001 C CNN
-	1    6450 5350
 	1    0    0    -1
 $EndComp
@@
 Wire Wire Line
 	6000 3750 6250 3750
+$Comp
+L MRDT_Connectors:Molex_SL_05 Conn?
+U 1 1 5FD25AC5
+P 6450 5450
+F 0 "Conn?" H 6578 5758 60  0000 L CNN
+F 1 "Molex_SL_05" H 6578 5652 60  0000 L CNN
+F 2 "" H 6450 5450 60  0001 C CNN
+F 3 "" H 6450 5450 60  0001 C CNN
+	1    6450 5450
+	1    0    0    -1
+$EndComp
+Text HLabel 6000 5400 0    50   Output ~ 0
+CurrentSenseHigh
+Wire Wire Line
+	6250 5400 6000 5400
 $EndSCHEMATC

Commit message: Started work on BOM
Parts:
- Conn2: renamed from Conn?; footprint (none) -> MRDT_Connectors:MOLEX_SL_05_Horizontal
Changed lines of the file:
@@
 EESchema Schematic File Version 4
-LIBS:12VBoard_2021_Rev1-cache
 EELAYER 30 0
 EELAYER END
@@
 	6000 3750 6250 3750
 $Comp
-L MRDT_Connectors:Molex_SL_05 Conn?
+L MRDT_Connectors:Molex_SL_05 Conn2
 U 1 1 5FD25AC5
 P 6450 5450
-F 0 "Conn?" H 6578 5758 60  0000 L CNN
+F 0 "Conn2" H 6578 5758 60  0000 L CNN
 F 1 "Molex_SL_05" H 6578 5652 60  0000 L CNN
-F 2 "" H 6450 5450 60  0001 C CNN
+F 2 "MRDT_Connectors:MOLEX_SL_05_Horizontal" H 6450 5450 60  0001 C CNN
 F 3 "" H 6450 5450 60  0001 C CNN
 	1    6450 5450

Commit message: Fixed problem
Connections:
- net CurrentSenseHigh renamed BuckCTL
Other:
- note added: "Buck CTL (Digital Write)\n"
- note removed: "Tiva 4 analog(current sense)/ \n7 toggles(digital write)"
Changed lines of the file:
@@
 $Descr A4 11693 8268
 encoding utf-8
-Sheet 7 8
+Sheet 3 8
 Title ""
 Date ""
@@
 Comment4 ""
 $EndDescr
-Text Notes 5650 3450 0    79   ~ 0
-Tiva 4 analog(current sense)/ \n7 toggles(digital write)
 Text HLabel 6000 5100 0    49   Input ~ 0
 AuxMountSense
@@
 	1    0    0    -1
 $EndComp
-Text HLabel 6000 5400 0    50   Output ~ 0
-CurrentSenseHigh
 Wire Wire Line
 	6250 5400 6000 5400
+Text HLabel 6000 5400 0    50   Input ~ 0
+BuckCTL
+Text Notes 6570 5430 0    50   ~ 0
+Buck CTL (Digital Write)\n
 $EndSCHEMATC

Commit message: Started Rev 2
Parts:
- Conn2: symbol MRDT_Connectors:Molex_SL_05 -> MRDT_Connectors:Molex_SL_04
Connections:
- net AuxMountCTL_Act: now also Conn1.1; no longer Conn1.4
- net AuxMountCTL_Log: now also Conn1.4; no longer Conn1.3
- net GimbalCTL_Act: now also Conn1.2; no longer Conn1.6
- net MultiMediaCTL_Log: now also Conn1.6; no longer Conn1.1
- net MultimediaCTL_Act: now also Conn1.3; no longer Conn1.2
- removed net BuckCTL: Conn2.5
Other:
- note added: "Ignore These"
- note removed: "Buck CTL (Digital Write)\n"
Changed lines of the file:
@@
 	1    0    0    -1
 $EndComp
-Text Notes 6575 3875 0    50   ~ 0
+Text Notes 9015 3705 0    50   ~ 0
 Multimedia Act CTL (Digital Write)
-Text Notes 6575 3775 0    50   ~ 0
+Text Notes 9015 3605 0    50   ~ 0
 Multimedia Log CTL (Digital Write)
-Text Notes 6575 4075 0    50   ~ 0
+Text Notes 9015 3905 0    50   ~ 0
 AuxMount Act CTL (Digital Write)
-Text Notes 6575 3975 0    50   ~ 0
+Text Notes 9015 3805 0    50   ~ 0
 AuxMount Log CTL (Digital Write)
-Text Notes 6575 4275 0    50   ~ 0
+Text Notes 9015 4105 0    50   ~ 0
 Gimbal Act CTL (Digital Write)
-Text Notes 6575 4175 0    50   ~ 0
+Text Notes 9015 4005 0    50   ~ 0
 Gimbal Log CTL (Digital Write)
-Text Notes 6575 4375 0    50   ~ 0
+Text Notes 9015 4205 0    50   ~ 0
 NavBoard CTL (Digital Write)
-Text Notes 6575 4475 0    50   ~ 0
+Text Notes 9015 4305 0    50   ~ 0
 Camera CTL (Digital Write)
-Text Notes 6575 4575 0    50   ~ 0
+Text Notes 9015 4405 0    50   ~ 0
 Extra CTL (Digitial Write)
-Text Notes 6575 4675 0    50   ~ 0
+Text Notes 9015 4500 0    50   ~ 0
 Drive  CTL (Digital Write)\n
-Text Notes 6575 5125 0    50   ~ 0
+Text Notes 9045 4905 0    50   ~ 0
 AuxMount Sense (Analog Read)
-Text Notes 6575 5025 0    50   ~ 0
+Text Notes 9045 4805 0    50   ~ 0
 Multimedia Sense (Analog Read)\n
-Text Notes 6575 5225 0    50   ~ 0
+Text Notes 9045 5005 0    50   ~ 0
 Gimbal Sense (Analog Read)
-Text Notes 6575 5325 0    50   ~ 0
+Text Notes 9045 5105 0    50   ~ 0
 Low Current Sense (Analog Read)
 Wire Wire Line
@@
 Wire Wire Line
 	6000 5300 6250 5300
-Text HLabel 6000 4050 0    49   Output ~ 0
+Text HLabel 6000 3750 0    49   Output ~ 0
 AuxMountCTL_Act
-Text HLabel 6000 4250 0    49   Output ~ 0
+Text HLabel 6000 3850 0    49   Output ~ 0
 GimbalCTL_Act
-Text HLabel 6000 3850 0    49   Output ~ 0
+Text HLabel 6000 3950 0    49   Output ~ 0
 MultimediaCTL_Act
 Wire Wire Line
@@
 Wire Wire Line
 	6000 4650 6250 4650
-Text HLabel 6000 3750 0    50   Output ~ 0
+Text HLabel 6000 4250 0    50   Output ~ 0
 MultiMediaCTL_Log
-Text HLabel 6000 3950 0    50   Output ~ 0
+Text HLabel 6000 4050 0    50   Output ~ 0
 AuxMountCTL_Log
 Text HLabel 6000 4150 0    50   Output ~ 0
@@
 	6000 3750 6250 3750
 $Comp
-L MRDT_Connectors:Molex_SL_05 Conn2
+L MRDT_Connectors:Molex_SL_04 Conn2
 U 1 1 5FD25AC5
-P 6450 5450
-F 0 "Conn2" H 6578 5758 60  0000 L CNN
-F 1 "Molex_SL_05" H 6578 5652 60  0000 L CNN
-F 2 "MRDT_Connectors:MOLEX_SL_05_Horizontal" H 6450 5450 60  0001 C CNN
-F 3 "" H 6450 5450 60  0001 C CNN
-	1    6450 5450
+P 6450 5350
+F 0 "Conn2" H 6578 5658 60  0000 L CNN
+F 1 "Molex_SL_05" H 6578 5552 60  0000 L CNN
+F 2 "MRDT_Connectors:MOLEX_SL_05_Horizontal" H 6450 5350 60  0001 C CNN
+F 3 "" H 6450 5350 60  0001 C CNN
+	1    6450 5350
 	1    0    0    -1
 $EndComp
-Wire Wire Line
-	6250 5400 6000 5400
-Text HLabel 6000 5400 0    50   Input ~ 0
-BuckCTL
-Text Notes 6570 5430 0    50   ~ 0
-Buck CTL (Digital Write)\n
+Text Notes 7530 3235 0    472  ~ 94
+Ignore These
 $EndSCHEMATC

Commit message: Rev 2 redone
in conclusion rev2=rev3 but its really rev12
Parts:
- Conn1: footprint MRDT_Connectors:MOLEX_SL_10_Horizontal -> MRDT_Connectors:MOLEX_SL_07_Vertical; symbol MRDT_Connectors:Molex_SL_10 -> MRDT_Connectors:Molex_SL_07
- Conn2: footprint MRDT_Connectors:MOLEX_SL_05_Horizontal -> MRDT_Connectors:MOLEX_SL_04_Vertical
Connections:
- net AuxMountCTL_Act is gone; now on net GimbalCTL_Act: Conn1.1
- net AuxMountCTL_Log is gone; now on net MultiMediaCTL_Log: Conn1.4
- net AuxMountSense is gone; now on net MultimediaSense: Conn2.2
- net CameraCTL: now also Conn1.5; no longer Conn1.8
- net DriveCTL: now also Conn1.7; no longer Conn1.10
- net ExtraCTL: now also Conn1.6; no longer Conn1.9
- net GimbalCTL_Act: no longer Conn1.2
- net GimbalCTL_Log: now also Conn1.3; no longer Conn1.5
- net MultiMediaCTL_Log: no longer Conn1.6
- net MultimediaCTL_Act: now also Conn1.2; no longer Conn1.3
- net MultimediaSense: no longer Conn2.1
- net NavBoardCTL: now also Conn2.1; no longer Conn1.7
Changed lines of the file:
@@
 $Descr A4 11693 8268
 encoding utf-8
-Sheet 3 8
+Sheet 3 7
 Title ""
 Date ""
@@
 $EndDescr
 Text HLabel 6000 5100 0    49   Input ~ 0
-AuxMountSense
-Text HLabel 6000 5000 0    49   Input ~ 0
 MultimediaSense
 Text HLabel 6000 5300 0    49   Input ~ 0
@@
 Text HLabel 6000 4450 0    49   Output ~ 0
 CameraCTL
-Text HLabel 6000 4350 0    49   Output ~ 0
-NavBoardCTL
 Text HLabel 6000 4550 0    49   Output ~ 0
 ExtraCTL
@@
 Text HLabel 6000 4650 0    50   Output ~ 0
 DriveCTL
-$Comp
-L MRDT_Connectors:Molex_SL_10 Conn1
-U 1 1 5FB5A813
-P 6450 4700
-F 0 "Conn1" H 6325 4550 60  0000 L CNN
-F 1 "Molex_SL_10" H 6175 4650 60  0000 L CNN
-F 2 "MRDT_Connectors:MOLEX_SL_10_Horizontal" H 6450 5200 60  0001 C CNN
-F 3 "" H 6450 5200 60  0001 C CNN
-	1    6450 4700
-	1    0    0    -1
-$EndComp
 Text Notes 9015 3705 0    50   ~ 0
 Multimedia Act CTL (Digital Write)
@@
 Low Current Sense (Analog Read)
 Wire Wire Line
-	6000 5000 6250 5000
-Wire Wire Line
 	6000 5100 6250 5100
 Wire Wire Line
@@
 Wire Wire Line
 	6000 5300 6250 5300
-Text HLabel 6000 3750 0    49   Output ~ 0
-AuxMountCTL_Act
-Text HLabel 6000 3850 0    49   Output ~ 0
+Text HLabel 6000 4050 0    49   Output ~ 0
 GimbalCTL_Act
-Text HLabel 6000 3950 0    49   Output ~ 0
-MultimediaCTL_Act
-Wire Wire Line
-	6000 4350 6250 4350
 Wire Wire Line
 	6000 4450 6250 4450
@@
 Wire Wire Line
 	6000 4650 6250 4650
+Text HLabel 6000 4350 0    50   Output ~ 0
+MultiMediaCTL_Log
 Text HLabel 6000 4250 0    50   Output ~ 0
-MultiMediaCTL_Log
-Text HLabel 6000 4050 0    50   Output ~ 0
-AuxMountCTL_Log
-Text HLabel 6000 4150 0    50   Output ~ 0
 GimbalCTL_Log
+Wire Wire Line
+	6000 4350 6250 4350
 Wire Wire Line
 	6000 4250 6250 4250
 Wire Wire Line
-	6000 4150 6250 4150
-Wire Wire Line
 	6000 4050 6250 4050
-Wire Wire Line
-	6000 3950 6250 3950
-Wire Wire Line
-	6000 3850 6250 3850
-Wire Wire Line
-	6000 3750 6250 3750
 $Comp
 L MRDT_Connectors:Molex_SL_04 Conn2
@@
 F 0 "Conn2" H 6578 5658 60  0000 L CNN
 F 1 "Molex_SL_05" H 6578 5552 60  0000 L CNN
-F 2 "MRDT_Connectors:MOLEX_SL_05_Horizontal" H 6450 5350 60  0001 C CNN
+F 2 "MRDT_Connectors:MOLEX_SL_04_Vertical" H 6450 5350 60  0001 C CNN
 F 3 "" H 6450 5350 60  0001 C CNN
 	1    6450 5350
@@
 Text Notes 7530 3235 0    472  ~ 94
 Ignore These
+Wire Wire Line
+	6000 4150 6250 4150
+Text HLabel 6000 4150 0    49   Output ~ 0
+MultimediaCTL_Act
+$Comp
+L MRDT_Connectors:Molex_SL_07 Conn1
+U 1 1 5FB5A813
+P 6450 4700
+F 0 "Conn1" H 6325 4550 60  0000 L CNN
+F 1 "Molex_SL_10" H 6175 4650 60  0000 L CNN
+F 2 "MRDT_Connectors:MOLEX_SL_07_Vertical" H 6450 5200 60  0001 C CNN
+F 3 "" H 6450 5200 60  0001 C CNN
+	1    6450 4700
+	1    0    0    -1
+$EndComp
+Wire Wire Line
+	6000 5000 6250 5000
+Text HLabel 6000 5000 0    49   Output ~ 0
+NavBoardCTL
 $EndSCHEMATC
