File: Hardware/12VBoard_2021_Rev1/Low Current Outputs.sch (KiCad schematic (older format))
At the start: 0 parts

Commit message: YELLED AT DAN WITHOUT HIM HERE
Parts:
- added C? (x5): 1000 uF, symbol Device:CP1
- added C? (x5): 100 uF, symbol Device:CP1
- added Conn? (x12): AndersonPP, symbol MRDT_Connectors:AndersonPP
- added D? (x5): 12V, Diode_SMD:D_0603_1608Metric_Pad1.05x0.95mm_HandSolder, symbol Device:D
- added L? (x5): 100 uH, Inductor_SMD:L_0603_1608Metric_Pad1.05x0.95mm_HandSolder, symbol Device:L
- added SW?: SW_SPDT, symbol Switch:SW_SPDT
- added U? (x5): LM2576D2TR4, MRDT_Devices:LM2576, symbol 12VBoard_2021_Rev1-rescue:LM2576D2TR4-MRDT_Devices
Connections:
- net labels added: +3.3V, GND
- wire segments 31 -> 215

Commit message: Ferite bead?
MERGE?????
Parts:
- added D? (x6): LED, symbol Device:LED
- added R? (x6): 1k, symbol Device:R
Connections:
- net labels added: 5V
- net labels removed: +3.3V
- wire segments 215 -> 210
Other:
- note added: "Green"
- moved on the sheet: Conn?A, Conn?B

Commit message: SHOCKKY :D
anthony mad
Parts:
- removed D? (x5): 12V, Diode_SMD:D_0603_1608Metric_Pad1.05x0.95mm_HandSolder, symbol Device:D
- added D? (x5): D_Schottky, symbol Device:D_Schottky
Connections:
- net GND: now also D?.2 (A), D?.2 (A), D?.2 (A), D?.2 (A), D?.2 (A)
- net at L?.1, U?.2 (OUTPUT): now also D?.1 (K) (x5)
Changed lines of the file:
@@
-$EndComp
-$Comp
-L Device:D D?
-U 1 1 5F850755
-P 4125 1450
-AR Path="/5F74F223/5F7D1238/5F850755" Ref="D?"  Part="1"
-AR Path="/5F74F223/5F7E1E8A/5F850755" Ref="D?"  Part="1"
-AR Path="/5F74F223/5F7D14F6/5F850755" Ref="D?"  Part="1"
-AR Path="/5F74F223/5F850755" Ref="D?"  Part="1"
-F 0 "D?" V 4079 1530 50  0000 L CNN
-F 1 "12V" V 4170 1530 50  0000 L CNN
-F 2 "Diode_SMD:D_0603_1608Metric_Pad1.05x0.95mm_HandSolder" H 4125 1450 50  0001 C CNN
-F 3 "~" H 4125 1450 50  0001 C CNN
-	1    4125 1450
-	0    1    1    0
 $EndComp
 $Comp
@@
 $EndComp
 $Comp
-L Device:D D?
-U 1 1 5F853A33
-P 4150 2725
-AR Path="/5F74F223/5F7D1238/5F853A33" Ref="D?"  Part="1"
-AR Path="/5F74F223/5F7E1E8A/5F853A33" Ref="D?"  Part="1"
-AR Path="/5F74F223/5F7D14F6/5F853A33" Ref="D?"  Part="1"
-AR Path="/5F74F223/5F853A33" Ref="D?"  Part="1"
-F 0 "D?" V 4104 2805 50  0000 L CNN
-F 1 "12V" V 4195 2805 50  0000 L CNN
-F 2 "Diode_SMD:D_0603_1608Metric_Pad1.05x0.95mm_HandSolder" H 4150 2725 50  0001 C CNN
-F 3 "~" H 4150 2725 50  0001 C CNN
-	1    4150 2725
-	0    1    1    0
-$EndComp
-$Comp
 L power:GND #PWR?
 U 1 1 5F853A3A
@@
 $EndComp
 $Comp
-L Device:D D?
-U 1 1 5F85809F
-P 4175 3975
-AR Path="/5F74F223/5F7D1238/5F85809F" Ref="D?"  Part="1"
-AR Path="/5F74F223/5F7E1E8A/5F85809F" Ref="D?"  Part="1"
-AR Path="/5F74F223/5F7D14F6/5F85809F" Ref="D?"  Part="1"
-AR Path="/5F74F223/5F85809F" Ref="D?"  Part="1"
-F 0 "D?" V 4129 4055 50  0000 L CNN
-F 1 "12V" V 4220 4055 50  0000 L CNN
-F 2 "Diode_SMD:D_0603_1608Metric_Pad1.05x0.95mm_HandSolder" H 4175 3975 50  0001 C CNN
-F 3 "~" H 4175 3975 50  0001 C CNN
-	1    4175 3975
-	0    1    1    0
-$EndComp
-$Comp
 L power:GND #PWR?
 U 1 1 5F8580A6
@@
 	4175 3750 4375 3750
 Wire Wire Line
-	4175 3750 4175 3825
-Wire Wire Line
 	4975 4125 4975 4175
 Wire Wire Line
@@
 $EndComp
 $Comp
-L Device:D D?
-U 1 1 5F85F736
-P 4225 5300
-AR Path="/5F74F223/5F7D1238/5F85F736" Ref="D?"  Part="1"
-AR Path="/5F74F223/5F7E1E8A/5F85F736" Ref="D?"  Part="1"
-AR Path="/5F74F223/5F7D14F6/5F85F736" Ref="D?"  Part="1"
-AR Path="/5F74F223/5F85F736" Ref="D?"  Part="1"
-F 0 "D?" V 4179 5380 50  0000 L CNN
-F 1 "12V" V 4270 5380 50  0000 L CNN
-F 2 "Diode_SMD:D_0603_1608Metric_Pad1.05x0.95mm_HandSolder" H 4225 5300 50  0001 C CNN
-F 3 "~" H 4225 5300 50  0001 C CNN
-	1    4225 5300
-	0    1    1    0
-$EndComp
-$Comp
 L power:GND #PWR?
 U 1 1 5F85F73D
@@
 $EndComp
 $Comp
-L Device:D D?
-U 1 1 5F86A2D3
-P 4275 6750
-AR Path="/5F74F223/5F7D1238/5F86A2D3" Ref="D?"  Part="1"
-AR Path="/5F74F223/5F7E1E8A/5F86A2D3" Ref="D?"  Part="1"
-AR Path="/5F74F223/5F7D14F6/5F86A2D3" Ref="D?"  Part="1"
-AR Path="/5F74F223/5F86A2D3" Ref="D?"  Part="1"
-F 0 "D?" V 4229 6830 50  0000 L CNN
-F 1 "12V" V 4320 6830 50  0000 L CNN
-F 2 "Diode_SMD:D_0603_1608Metric_Pad1.05x0.95mm_HandSolder" H 4275 6750 50  0001 C CNN
-F 3 "~" H 4275 6750 50  0001 C CNN
-	1    4275 6750
-	0    1    1    0
-$EndComp
-$Comp
 L power:GND #PWR?
 U 1 1 5F86A2DA
@@
 Wire Wire Line
 	6425 5525 6425 5700
+$Comp
+L Device:D_Schottky D?
+U 1 1 5F88AAB0
+P 4125 1450
+F 0 "D?" V 4079 1530 50  0000 L CNN
+F 1 "D_Schottky" V 4170 1530 50  0000 L CNN
+F 2 "" H 4125 1450 50  0001 C CNN
+F 3 "~" H 4125 1450 50  0001 C CNN
+	1    4125 1450
+	0    1    1    0
+$EndComp
+$Comp
+L Device:D_Schottky D?
+U 1 1 5F88BCE9
+P 4150 2725
+F 0 "D?" V 4104 2805 50  0000 L CNN
+F 1 "D_Schottky" V 4195 2805 50  0000 L CNN
+F 2 "" H 4150 2725 50  0001 C CNN
+F 3 "~" H 4150 2725 50  0001 C CNN
+	1    4150 2725
+	0    1    1    0
+$EndComp
+$Comp
+L Device:D_Schottky D?
+U 1 1 5F88D34D
+P 4175 3975
+F 0 "D?" V 4129 4055 50  0000 L CNN
+F 1 "D_Schottky" V 4220 4055 50  0000 L CNN
+F 2 "" H 4175 3975 50  0001 C CNN
+F 3 "~" H 4175 3975 50  0001 C CNN
+	1    4175 3975
+	0    1    1    0
+$EndComp
+Wire Wire Line
+	4175 3750 4175 3825
+$Comp
+L Device:D_Schottky D?
+U 1 1 5F88F5BA
+P 4225 5300
+F 0 "D?" V 4179 5380 50  0000 L CNN
+F 1 "D_Schottky" V 4270 5380 50  0000 L CNN
+F 2 "" H 4225 5300 50  0001 C CNN
+F 3 "~" H 4225 5300 50  0001 C CNN
+	1    4225 5300
+	0    1    1    0
+$EndComp
+$Comp
+L Device:D_Schottky D?
+U 1 1 5F88FCBF
+P 4275 6750
+F 0 "D?" V 4229 6830 50  0000 L CNN
+F 1 "D_Schottky" V 4320 6830 50  0000 L CNN
+F 2 "" H 4275 6750 50  0001 C CNN
+F 3 "~" H 4275 6750 50  0001 C CNN
+	1    4275 6750
+	0    1    1    0
+$EndComp
 $EndSCHEMATC

Commit message: finished low current
Parts:
- removed D?: LED, symbol Device:LED
- removed R?: 1k, symbol Device:R
- added R?: 5m, symbol Device:R
- added U?: INA198, Package_TO_SOT_SMD:SOT-23-5, symbol Amplifier_Current:INA198
Connections:
- net 5V: now also U?.3 (V+)
- net GND: now also U?.2 (GND)
- net at C?.1, L?.2, U?.4 (FEEDBACK): now also R?.1, U?.5 (-); no longer Conn?.2 (V+Log), Conn?.2 (V+Log), R?.1
- new net: Conn?.2 (V+Log), Conn?.2 (V+Log), R?.1, R?.2, U?.4 (+)
- new net CurrentSense: U?.1
Other:
- moved on the sheet: Conn?A, Conn?B, D?, R?

Commit message: High current
Fisnished adding labes/tags
Parts:
- R?: value 5m -> 25m
Changed lines of the file:
@@
 	1    0    0    -1
 $EndComp
-$Comp
-L power:GND #PWR?
-U 1 1 5F853A46
-P 2225 2375
-AR Path="/5F74F223/5F7D1238/5F853A46" Ref="#PWR?"  Part="1"
-AR Path="/5F74F223/5F7D14F6/5F853A46" Ref="#PWR?"  Part="1"
-AR Path="/5F74F223/5F853A46" Ref="#PWR?"  Part="1"
-F 0 "#PWR?" H 2225 2125 50  0001 C CNN
-F 1 "GND" H 2230 2202 50  0000 C CNN
-F 2 "" H 2225 2375 50  0001 C CNN
-F 3 "" H 2225 2375 50  0001 C CNN
-	1    2225 2375
-	1    0    0    -1
-$EndComp
-Wire Wire Line
-	2625 2650 2500 2650
 Wire Wire Line
 	5500 2825 5500 2925
@@
 Wire Wire Line
 	2250 1225 2600 1225
-Wire Wire Line
-	2625 2500 2500 2500
-Wire Wire Line
-	2625 2350 2425 2350
-Wire Wire Line
-	2225 2350 2225 2375
-Wire Wire Line
-	2425 2500 2425 2350
-Connection ~ 2425 2350
-Wire Wire Line
-	2425 2350 2225 2350
-Wire Wire Line
-	2500 2650 2500 2500
-Connection ~ 2500 2500
-Wire Wire Line
-	2500 2500 2425 2500
 $Comp
 L MRDT_Connectors:AndersonPP Conn?
@@
 AR Path="/5F74F223/5F928AA0" Ref="R?"  Part="1"
 F 0 "R?" V 5893 7250 50  0000 C CNN
-F 1 "5m" V 5984 7250 50  0000 C CNN
+F 1 "25m" V 5984 7250 50  0000 C CNN
 F 2 "" V 6030 7250 50  0001 C CNN
 F 3 "~" H 6100 7250 50  0001 C CNN
@@
 Wire Wire Line
 	9000 6250 9000 6425
+Wire Wire Line
+	2500 2500 2425 2500
+Wire Wire Line
+	2500 2650 2500 2500
+Wire Wire Line
+	2425 2350 2225 2350
+Wire Wire Line
+	2425 2500 2425 2350
+Wire Wire Line
+	2225 2350 2225 2375
+Connection ~ 2425 2350
+Wire Wire Line
+	2625 2350 2425 2350
+Connection ~ 2500 2500
+Wire Wire Line
+	2625 2500 2500 2500
+Wire Wire Line
+	2625 2650 2500 2650
+$Comp
+L power:GND #PWR?
+U 1 1 5F853A46
+P 2225 2375
+AR Path="/5F74F223/5F7D1238/5F853A46" Ref="#PWR?"  Part="1"
+AR Path="/5F74F223/5F7D14F6/5F853A46" Ref="#PWR?"  Part="1"
+AR Path="/5F74F223/5F853A46" Ref="#PWR?"  Part="1"
+F 0 "#PWR?" H 2225 2125 50  0001 C CNN
+F 1 "GND" H 2230 2202 50  0000 C CNN
+F 2 "" H 2225 2375 50  0001 C CNN
+F 3 "" H 2225 2375 50  0001 C CNN
+	1    2225 2375
+	1    0    0    -1
+$EndComp
 $EndSCHEMATC

Commit message: Added Testpoints
Parts:
- added TP? (x4): TestPoint, symbol Connector:TestPoint
Connections:
- net CameraToggle: now also TP?.1
- net CurrentSense: now also TP?.1
- net GimbalToggle: now also TP?.1
- net NavToggle: now also TP?.1
Changed lines of the file:
@@
 GimbalToggle
 Wire Wire Line
-	2350 5075 2700 5075
+	2350 5075 2450 5075
 Text HLabel 2300 3750 0    79   Input ~ 0
 NavToggle
 Wire Wire Line
-	2300 3750 2650 3750
+	2300 3750 2450 3750
 Text HLabel 2250 1225 0    79   Input ~ 0
 CameraToggle
 Wire Wire Line
-	2250 1225 2600 1225
+	2250 1225 2400 1225
 $Comp
 L MRDT_Connectors:AndersonPP Conn?
@@
 	1    0    0    -1
 $EndComp
+$Comp
+L Connector:TestPoint TP?
+U 1 1 5F90B4C6
+P 6100 6000
+F 0 "TP?" H 6158 6118 50  0000 L CNN
+F 1 "TestPoint" H 6158 6027 50  0000 L CNN
+F 2 "" H 6300 6000 50  0001 C CNN
+F 3 "~" H 6300 6000 50  0001 C CNN
+	1    6100 6000
+	1    0    0    -1
+$EndComp
+Wire Wire Line
+	6100 6100 6100 6000
+Connection ~ 6100 6100
+$Comp
+L Connector:TestPoint TP?
+U 1 1 5F9264D0
+P 2450 5200
+F 0 "TP?" H 2508 5318 50  0000 L CNN
+F 1 "TestPoint" H 2508 5227 50  0000 L CNN
+F 2 "" H 2650 5200 50  0001 C CNN
+F 3 "~" H 2650 5200 50  0001 C CNN
+	1    2450 5200
+	-1   0    0    1
+$EndComp
+$Comp
+L Connector:TestPoint TP?
+U 1 1 5F933AA4
+P 2450 3900
+F 0 "TP?" H 2508 4018 50  0000 L CNN
+F 1 "TestPoint" H 2508 3927 50  0000 L CNN
+F 2 "" H 2650 3900 50  0001 C CNN
+F 3 "~" H 2650 3900 50  0001 C CNN
+	1    2450 3900
+	-1   0    0    1
+$EndComp
+$Comp
+L Connector:TestPoint TP?
+U 1 1 5F940F94
+P 2400 1350
+F 0 "TP?" H 2458 1468 50  0000 L CNN
+F 1 "TestPoint" H 2458 1377 50  0000 L CNN
+F 2 "" H 2600 1350 50  0001 C CNN
+F 3 "~" H 2600 1350 50  0001 C CNN
+	1    2400 1350
+	-1   0    0    1
+$EndComp
+Wire Wire Line
+	2450 3900 2450 3750
+Connection ~ 2450 3750
+Wire Wire Line
+	2450 3750 2650 3750
+Wire Wire Line
+	2450 5075 2450 5200
+Connection ~ 2450 5075
+Wire Wire Line
+	2450 5075 2700 5075
+Wire Wire Line
+	2400 1350 2400 1225
+Connection ~ 2400 1225
+Wire Wire Line
+	2400 1225 2600 1225
 $EndSCHEMATC

Commit message: reviewed
review
Parts:
- removed C? (x5): 100 uF, symbol Device:CP1
- added C? (x5): 100uF, symbol Device:C_Small
- R? (x5): value 1k -> 1.2k
Connections:
- net 5V: no longer SW?.1 (A)
- net GND: now also C?.2, C?.2, C?.2, C?.2, C?.2
- net PackVoltage: now also C?.1, C?.1, C?.1, C?.1, C?.1
- new net ExtraToggle: SW?.1 (A)
Changed lines of the file:
@@
 $Descr A4 11693 8268
 encoding utf-8
-Sheet 4 8
+Sheet 4 7
 Title ""
 Date ""
@@
 	2475 1375 2475 1675
 Wire Wire Line
-	5475 1550 5475 1650
-$Comp
-L Device:CP1 C?
-U 1 1 5F850792
-P 5475 1400
-AR Path="/5F74F223/5F7D1238/5F850792" Ref="C?"  Part="1"
-AR Path="/5F74F223/5F7E1E8A/5F850792" Ref="C?"  Part="1"
-AR Path="/5F74F223/5F7D14F6/5F850792" Ref="C?"  Part="1"
-AR Path="/5F74F223/5F850792" Ref="C?"  Part="1"
-F 0 "C?" V 5250 1450 50  0000 R CNN
-F 1 "100 uF" V 5325 1525 50  0000 R CNN
-F 2 "" H 5475 1400 50  0001 C CNN
-F 3 "~" H 5475 1400 50  0001 C CNN
-	1    5475 1400
-	1    0    0    -1
-$EndComp
-Wire Wire Line
 	5475 1075 5475 1250
 Wire Wire Line
@@
 $EndComp
 Wire Wire Line
-	5500 2825 5500 2925
-$Comp
-L Device:CP1 C?
-U 1 1 5F853A70
-P 5500 2675
-AR Path="/5F74F223/5F7D1238/5F853A70" Ref="C?"  Part="1"
-AR Path="/5F74F223/5F7E1E8A/5F853A70" Ref="C?"  Part="1"
-AR Path="/5F74F223/5F7D14F6/5F853A70" Ref="C?"  Part="1"
-AR Path="/5F74F223/5F853A70" Ref="C?"  Part="1"
-F 0 "C?" V 5275 2725 50  0000 R CNN
-F 1 "100 uF" V 5350 2800 50  0000 R CNN
-F 2 "" H 5500 2675 50  0001 C CNN
-F 3 "~" H 5500 2675 50  0001 C CNN
-	1    5500 2675
-	1    0    0    -1
-$EndComp
-Wire Wire Line
 	5500 2350 5500 2525
 Wire Wire Line
@@
 	2525 3900 2525 4200
 Wire Wire Line
-	5525 4075 5525 4175
-$Comp
-L Device:CP1 C?
-U 1 1 5F8580DC
-P 5525 3925
-AR Path="/5F74F223/5F7D1238/5F8580DC" Ref="C?"  Part="1"
-AR Path="/5F74F223/5F7E1E8A/5F8580DC" Ref="C?"  Part="1"
-AR Path="/5F74F223/5F7D14F6/5F8580DC" Ref="C?"  Part="1"
-AR Path="/5F74F223/5F8580DC" Ref="C?"  Part="1"
-F 0 "C?" V 5300 3975 50  0000 R CNN
-F 1 "100 uF" V 5375 4050 50  0000 R CNN
-F 2 "" H 5525 3925 50  0001 C CNN
-F 3 "~" H 5525 3925 50  0001 C CNN
-	1    5525 3925
-	1    0    0    -1
-$EndComp
-Wire Wire Line
 	5525 3600 5525 3775
 Wire Wire Line
@@
 	2575 5225 2575 5525
 Wire Wire Line
-	5575 5400 5575 5500
-$Comp
-L Device:CP1 C?
-U 1 1 5F85F773
-P 5575 5250
-AR Path="/5F74F223/5F7D1238/5F85F773" Ref="C?"  Part="1"
-AR Path="/5F74F223/5F7E1E8A/5F85F773" Ref="C?"  Part="1"
-AR Path="/5F74F223/5F7D14F6/5F85F773" Ref="C?"  Part="1"
-AR Path="/5F74F223/5F85F773" Ref="C?"  Part="1"
-F 0 "C?" V 5350 5300 50  0000 R CNN
-F 1 "100 uF" V 5425 5375 50  0000 R CNN
-F 2 "" H 5575 5250 50  0001 C CNN
-F 3 "~" H 5575 5250 50  0001 C CNN
-	1    5575 5250
-	1    0    0    -1
-$EndComp
-Wire Wire Line
 	5575 4925 5575 5100
 Wire Wire Line
@@
 	2625 6675 2625 6975
 Wire Wire Line
-	5625 6850 5625 6950
-$Comp
-L Device:CP1 C?
-U 1 1 5F86A310
-P 5625 6700
-AR Path="/5F74F223/5F7D1238/5F86A310" Ref="C?"  Part="1"
-AR Path="/5F74F223/5F7E1E8A/5F86A310" Ref="C?"  Part="1"
-AR Path="/5F74F223/5F7D14F6/5F86A310" Ref="C?"  Part="1"
-AR Path="/5F74F223/5F86A310" Ref="C?"  Part="1"
-F 0 "C?" V 5400 6750 50  0000 R CNN
-F 1 "100 uF" V 5475 6825 50  0000 R CNN
-F 2 "" H 5625 6700 50  0001 C CNN
-F 3 "~" H 5625 6700 50  0001 C CNN
-	1    5625 6700
-	1    0    0    -1
-$EndComp
-Wire Wire Line
 	5625 6375 5625 6550
 Wire Wire Line
@@
 Wire Wire Line
 	6975 1475 7050 1475
-Text HLabel 1350 6250 1    50   Input ~ 0
-5V
+Text HLabel 1350 6250 0    50   Input ~ 0
+ExtraToggle
 Connection ~ 6425 1850
 Wire Wire Line
@@
 AR Path="/5F74F223/5FA89BE6" Ref="R?"  Part="1"
 F 0 "R?" H 6495 5421 50  0000 L CNN
-F 1 "1k" H 6495 5330 50  0000 L CNN
+F 1 "1.2k" H 6495 5330 50  0000 L CNN
 F 2 "" V 6355 5375 50  0001 C CNN
 F 3 "~" H 6425 5375 50  0001 C CNN
@@
 AR Path="/5F74F223/5FA95394" Ref="R?"  Part="1"
 F 0 "R?" H 6495 4121 50  0000 L CNN
-F 1 "1k" H 6495 4030 50  0000 L CNN
+F 1 "1.2k" H 6495 4030 50  0000 L CNN
 F 2 "" V 6355 4075 50  0001 C CNN
 F 3 "~" H 6425 4075 50  0001 C CNN
@@
 AR Path="/5F74F223/5FAA0D2F" Ref="R?"  Part="1"
 F 0 "R?" H 6495 2821 50  0000 L CNN
-F 1 "1k" H 6495 2730 50  0000 L CNN
+F 1 "1.2k" H 6495 2730 50  0000 L CNN
 F 2 "" V 6355 2775 50  0001 C CNN
 F 3 "~" H 6425 2775 50  0001 C CNN
@@
 AR Path="/5F74F223/5FAACC52" Ref="R?"  Part="1"
 F 0 "R?" H 6495 1521 50  0000 L CNN
-F 1 "1k" H 6495 1430 50  0000 L CNN
+F 1 "1.2k" H 6495 1430 50  0000 L CNN
 F 2 "" V 6355 1475 50  0001 C CNN
 F 3 "~" H 6425 1475 50  0001 C CNN
@@
 AR Path="/5F74F223/5F8BCD25" Ref="R?"  Part="1"
 F 0 "R?" H 6695 6771 50  0000 L CNN
-F 1 "1k" H 6695 6680 50  0000 L CNN
+F 1 "1.2k" H 6695 6680 50  0000 L CNN
 F 2 "" V 6555 6725 50  0001 C CNN
 F 3 "~" H 6625 6725 50  0001 C CNN
@@
 Wire Wire Line
 	2400 1225 2600 1225
+$Comp
+L Device:C_Small C?
+U 1 1 5F8CDA71
+P 5475 1350
+F 0 "C?" H 5567 1396 50  0000 L CNN
+F 1 "100uF" H 5567 1305 50  0000 L CNN
+F 2 "" H 5475 1350 50  0001 C CNN
+F 3 "~" H 5475 1350 50  0001 C CNN
+	1    5475 1350
+	1    0    0    -1
+$EndComp
+Wire Wire Line
+	5475 1450 5475 1650
+$Comp
+L Device:C_Small C?
+U 1 1 5F8DCAFB
+P 5500 2625
+F 0 "C?" H 5592 2671 50  0000 L CNN
+F 1 "100uF" H 5592 2580 50  0000 L CNN
+F 2 "" H 5500 2625 50  0001 C CNN
+F 3 "~" H 5500 2625 50  0001 C CNN
+	1    5500 2625
+	1    0    0    -1
+$EndComp
+$Comp
+L Device:C_Small C?
+U 1 1 5F8DCE58
+P 5525 3875
+F 0 "C?" H 5617 3921 50  0000 L CNN
+F 1 "100uF" H 5617 3830 50  0000 L CNN
+F 2 "" H 5525 3875 50  0001 C CNN
+F 3 "~" H 5525 3875 50  0001 C CNN
+	1    5525 3875
+	1    0    0    -1
+$EndComp
+$Comp
+L Device:C_Small C?
+U 1 1 5F8DD1A5
+P 5575 5200
+F 0 "C?" H 5667 5246 50  0000 L CNN
+F 1 "100uF" H 5667 5155 50  0000 L CNN
+F 2 "" H 5575 5200 50  0001 C CNN
+F 3 "~" H 5575 5200 50  0001 C CNN
+	1    5575 5200
+	1    0    0    -1
+$EndComp
+$Comp
+L Device:C_Small C?
+U 1 1 5F8DD4B6
+P 5625 6650
+F 0 "C?" H 5400 6675 50  0000 L CNN
+F 1 "100uF" H 5325 6575 50  0000 L CNN
+F 2 "" H 5625 6650 50  0001 C CNN
+F 3 "~" H 5625 6650 50  0001 C CNN
+	1    5625 6650
+	1    0    0    -1
+$EndComp
+Wire Wire Line
+	5625 6750 5625 6950
+Wire Wire Line
+	5575 5300 5575 5500
+Wire Wire Line
+	5525 3975 5525 4175
+Wire Wire Line
+	5500 2725 5500 2925
 $EndSCHEMATC
