File: Hardware/12VBoard_2021_Rev1/Low Current Outputs.sch (KiCad schematic (older format))
At the start: 48 parts, among them U14 LM2576S-12/NOPB, U2 INA198, U3 LM2576S-12/NOPB, U4 LM2576S-12/NOPB, U5 LM2576S-12/NOPB, U6 LM2576S-12/NOPB

Commit message: Worked on layout
Low current bucks grouped with their componets
Parts:
- C3, C4, C43, C5, C6: footprint Capacitor_THT:CP_Axial_L20.0mm_D10.0mm_P26.00mm_Horizontal -> Capacitor_THT:CP_Radial_D10.0mm_P5.00mm
Changed lines of the file:
@@
 EESchema Schematic File Version 4
-LIBS:12VBoard_2021_Rev1-cache
 EELAYER 30 0
 EELAYER END
@@
 F 0 "C3" V 4700 1400 50  0000 L CNN
 F 1 "1000 uF" V 4775 1325 50  0000 L CNN
-F 2 "Capacitor_THT:CP_Axial_L20.0mm_D10.0mm_P26.00mm_Horizontal" H 4925 1450 50  0001 C CNN
+F 2 "Capacitor_THT:CP_Radial_D10.0mm_P5.00mm" H 4925 1450 50  0001 C CNN
 F 3 "~" H 4925 1450 50  0001 C CNN
 	1    4925 1450
@@
 F 0 "C4" V 4725 2675 50  0000 L CNN
 F 1 "1000 uF" V 4800 2600 50  0000 L CNN
-F 2 "Capacitor_THT:CP_Axial_L20.0mm_D10.0mm_P26.00mm_Horizontal" H 4950 2725 50  0001 C CNN
+F 2 "Capacitor_THT:CP_Radial_D10.0mm_P5.00mm" H 4950 2725 50  0001 C CNN
 F 3 "~" H 4950 2725 50  0001 C CNN
 	1    4950 2725
@@
 F 0 "C5" V 4750 3925 50  0000 L CNN
 F 1 "1000 uF" V 4825 3850 50  0000 L CNN
-F 2 "Capacitor_THT:CP_Axial_L20.0mm_D10.0mm_P26.00mm_Horizontal" H 4975 3975 50  0001 C CNN
+F 2 "Capacitor_THT:CP_Radial_D10.0mm_P5.00mm" H 4975 3975 50  0001 C CNN
 F 3 "~" H 4975 3975 50  0001 C CNN
 	1    4975 3975
@@
 F 0 "C6" V 4850 5090 50  0000 L CNN
 F 1 "1000 uF" V 4925 5015 50  0000 L CNN
-F 2 "Capacitor_THT:CP_Axial_L20.0mm_D10.0mm_P26.00mm_Horizontal" H 5075 5140 50  0001 C CNN
+F 2 "Capacitor_THT:CP_Radial_D10.0mm_P5.00mm" H 5075 5140 50  0001 C CNN
 F 3 "~" H 5075 5140 50  0001 C CNN
 	1    5075 5140
@@
 F 0 "C43" V 4650 6330 50  0000 L CNN
 F 1 "1000 uF" V 4725 6255 50  0000 L CNN
-F 2 "Capacitor_THT:CP_Axial_L20.0mm_D10.0mm_P26.00mm_Horizontal" H 4875 6380 50  0001 C CNN
+F 2 "Capacitor_THT:CP_Radial_D10.0mm_P5.00mm" H 4875 6380 50  0001 C CNN
 F 3 "~" H 4875 6380 50  0001 C CNN
 	1    4875 6380
