File: Hardware/12VBoard_2021_Rev1/Low Current Outputs.sch (KiCad schematic (older format))
At the start: 55 parts, among them Q10 IRLML2060, Q11 IRLML2060, Q12 IRLML2060, Q13 IRLML2060, U14 LT1910, U15 LT1910, U16 LT1910, U17 LT1910, U2 INA198, U4 LM2576S-12/NOPB, U9 OKI

Commit message: Started work on BOM
Parts:
- R3: footprint Package_TO_SOT_THT:TO-126-2_Vertical -> Resistor_SMD:R_1206_3216Metric_Pad1.42x1.75mm_HandSolder
Changed lines of the file:
@@
 EESchema Schematic File Version 4
-LIBS:12VBoard_2021_Rev1-cache
 EELAYER 30 0
 EELAYER END
@@
 F 0 "R3" V 1118 7275 50  0000 C CNN
 F 1 "50m" V 1209 7275 50  0000 C CNN
-F 2 "Package_TO_SOT_THT:TO-126-2_Vertical" V 1255 7275 50  0001 C CNN
+F 2 "Resistor_SMD:R_1206_3216Metric_Pad1.42x1.75mm_HandSolder" V 1255 7275 50  0001 C CNN
 F 3 "~" H 1325 7275 50  0001 C CNN
 	1    1325 7275

Commit message: Discovered problems, will fix on next pushes
Parts:
- R3: value 50m -> 20m
Changed lines of the file:
@@
 AR Path="/5F74F223/5FDB0B31" Ref="C45"  Part="1"
 F 0 "C45" H 4825 2800 50  0000 L CNN
-F 1 "10uF" H 4500 2700 50  0000 L CNN
+F 1 "10uF" H 4780 2670 50  0000 L CNN
 F 2 "Capacitor_THT:CP_Radial_D5.0mm_P2.00mm" H 5000 2750 50  0001 C CNN
 F 3 "~" H 5000 2750 50  0001 C CNN
@@
 AR Path="/5F74F223/5F8C9CDB" Ref="R3"  Part="1"
 F 0 "R3" V 1118 7275 50  0000 C CNN
-F 1 "50m" V 1209 7275 50  0000 C CNN
+F 1 "20m" V 1209 7275 50  0000 C CNN
 F 2 "Resistor_SMD:R_1206_3216Metric_Pad1.42x1.75mm_HandSolder" V 1255 7275 50  0001 C CNN
 F 3 "~" H 1325 7275 50  0001 C CNN
