File: Hardware/12VBoard_2021_Rev1/Gimbal.sch (KiCad schematic (older format))
At the start: 27 parts, among them Q6 2N7000, Q7 2N7000, U12 LM5116, U13 INA198

Commit message: Finished Footprint Assignment
added footprint for switch and finished footprint assigning aslwell as changeing low current current sense resistor to 50 m ohms.
Parts:
- R33: footprint (none) -> Resistor_SMD:R_2512_6332Metric_Pad1.52x3.35mm_HandSolder
Changed lines of the file:
@@
 F 0 "R33" V 3193 3550 50  0000 C CNN
 F 1 "50m" V 3284 3550 50  0000 C CNN
-F 2 "" V 3330 3550 50  0001 C CNN
+F 2 "Resistor_SMD:R_2512_6332Metric_Pad1.52x3.35mm_HandSolder" V 3330 3550 50  0001 C CNN
 F 3 "~" H 3400 3550 50  0001 C CNN
 	1    3400 3550

Commit message: Added Logic power circuits (High)
Added three smaller bucks for high current logic power and seprated acuation and logic pp
Parts:
- added C?: 100uF, Capacitor_SMD:C_0603_1608Metric_Pad1.05x0.95mm_HandSolder, symbol Device:C_Small
- added C?: 1000 uF, Capacitor_THT:CP_Axial_L20.0mm_D10.0mm_P26.00mm_Horizontal, symbol Device:CP1
- added D?: D_Schottky, Diode_SMD:D_0603_1608Metric_Pad1.05x0.95mm_HandSolder, symbol Device:D_Schottky
- added D?: Gimbal Logic Green, Diode_SMD:D_0603_1608Metric_Pad1.05x0.95mm_HandSolder, symbol Device:LED
- added L?: 100 uH, Inductor_SMD:L_0603_1608Metric_Pad1.05x0.95mm_HandSolder, symbol Device:L
- added R?: 1.2k, Resistor_SMD:R_0603_1608Metric_Pad0.98x0.95mm_HandSolder, symbol Device:R
- added TP?: TestPoint, TestPoint:TestPoint_Pad_2.5x2.5mm, symbol Connector:TestPoint
- added U?: LM2576S-12/NOPB, MRDT_Devices:LM2576, symbol 12VBoard_2021_Rev1-rescue:LM2576D2TR4-MRDT_Devices
- D18: value LED -> Gimbal Acuation Gree
Connections:
- net labels added: 12V3AGimbalLogic
- wire segments 116 -> 150

Commit message: Layout Started
Board dimensions
Parts:
- gave numbers to parts that had none: 8
Changed lines of the file:
@@
 $Descr A4 11693 8268
 encoding utf-8
-Sheet 8 8
+Sheet 7 8
 Title ""
 Date ""
@@
 P 6525 1425
 AR Path="/5F74F223/5FACC5D4" Ref="TP?"  Part="1"
-AR Path="/5F74F36B/5F971CD6/5FACC5D4" Ref="TP?"  Part="1"
-F 0 "TP?" H 6583 1543 50  0000 L CNN
+AR Path="/5F74F36B/5F971CD6/5FACC5D4" Ref="TP10"  Part="1"
+F 0 "TP10" H 6583 1543 50  0000 L CNN
 F 1 "TestPoint" H 6583 1452 50  0000 L CNN
 F 2 "TestPoint:TestPoint_Pad_2.5x2.5mm" H 6725 1425 50  0001 C CNN
@@
 P 9650 1425
 AR Path="/5F74F223/5FACC5E1" Ref="C?"  Part="1"
-AR Path="/5F74F36B/5F971CD6/5FACC5E1" Ref="C?"  Part="1"
-F 0 "C?" H 9425 1450 50  0000 L CNN
+AR Path="/5F74F36B/5F971CD6/5FACC5E1" Ref="C48"  Part="1"
+F 0 "C48" H 9425 1450 50  0000 L CNN
 F 1 "100uF" H 9350 1350 50  0000 L CNN
 F 2 "Capacitor_SMD:C_0603_1608Metric_Pad1.05x0.95mm_HandSolder" H 9650 1425 50  0001 C CNN
@@
 P 8300 1525
 AR Path="/5F74F223/5FACC5E7" Ref="D?"  Part="1"
-AR Path="/5F74F36B/5F971CD6/5FACC5E7" Ref="D?"  Part="1"
-F 0 "D?" V 8254 1605 50  0000 L CNN
+AR Path="/5F74F36B/5F971CD6/5FACC5E7" Ref="D23"  Part="1"
+F 0 "D23" V 8254 1605 50  0000 L CNN
 F 1 "D_Schottky" V 8345 1605 50  0000 L CNN
 F 2 "Diode_SMD:D_0603_1608Metric_Pad1.05x0.95mm_HandSolder" H 8300 1525 50  0001 C CNN
@@
 AR Path="/5F74F223/5F7D14F6/5FACC604" Ref="#PWR?"  Part="1"
 AR Path="/5F74F223/5FACC604" Ref="#PWR?"  Part="1"
-AR Path="/5F74F36B/5F971CD6/5FACC604" Ref="#PWR?"  Part="1"
-F 0 "#PWR?" H 6650 1500 50  0001 C CNN
+AR Path="/5F74F36B/5F971CD6/5FACC604" Ref="#PWR090"  Part="1"
+F 0 "#PWR090" H 6650 1500 50  0001 C CNN
 F 1 "GND" H 6655 1577 50  0000 C CNN
 F 2 "" H 6650 1750 50  0001 C CNN
@@
 AR Path="/5F74F223/5F7D14F6/5FACC60D" Ref="#PWR?"  Part="1"
 AR Path="/5F74F223/5FACC60D" Ref="#PWR?"  Part="1"
-AR Path="/5F74F36B/5F971CD6/5FACC60D" Ref="#PWR?"  Part="1"
-F 0 "#PWR?" H 6675 775 50  0001 C CNN
+AR Path="/5F74F36B/5F971CD6/5FACC60D" Ref="#PWR091"  Part="1"
+F 0 "#PWR091" H 6675 775 50  0001 C CNN
 F 1 "GND" H 6680 852 50  0000 C CNN
 F 2 "" H 6675 1025 50  0001 C CNN
@@
 AR Path="/5FACC613" Ref="U?"  Part="1"
 AR Path="/5F74F223/5FACC613" Ref="U?"  Part="1"
-AR Path="/5F74F36B/5F971CD6/5FACC613" Ref="U?"  Part="1"
-F 0 "U?" H 7275 1775 50  0000 C CNN
+AR Path="/5F74F36B/5F971CD6/5FACC613" Ref="U16"  Part="1"
+F 0 "U16" H 7275 1775 50  0000 C CNN
 F 1 "LM2576S-12/NOPB" H 7275 1684 50  0000 C CNN
 F 2 "MRDT_Devices:LM2576" H 7275 1800 50  0001 C CNN
@@
 AR Path="/5F74F223/5F7D14F6/5FACC619" Ref="#PWR?"  Part="1"
 AR Path="/5F74F223/5FACC619" Ref="#PWR?"  Part="1"
-AR Path="/5F74F36B/5F971CD6/5FACC619" Ref="#PWR?"  Part="1"
-F 0 "#PWR?" H 8700 1525 50  0001 C CNN
+AR Path="/5F74F36B/5F971CD6/5FACC619" Ref="#PWR092"  Part="1"
+F 0 "#PWR092" H 8700 1525 50  0001 C CNN
 F 1 "GND" H 8700 1625 50  0000 C CNN
 F 2 "" H 8700 1775 50  0001 C CNN
@@
 AR Path="/5F74F223/5F7D14F6/5FACC61F" Ref="C?"  Part="1"
 AR Path="/5F74F223/5FACC61F" Ref="C?"  Part="1"
-AR Path="/5F74F36B/5F971CD6/5FACC61F" Ref="C?"  Part="1"
-F 0 "C?" V 8875 1475 50  0000 L CNN
+AR Path="/5F74F36B/5F971CD6/5FACC61F" Ref="C47"  Part="1"
+F 0 "C47" V 8875 1475 50  0000 L CNN
 F 1 "1000 uF" V 8950 1400 50  0000 L CNN
 F 2 "Capacitor_THT:CP_Axial_L20.0mm_D10.0mm_P26.00mm_Horizontal" H 9100 1525 50  0001 C CNN
@@
 AR Path="/5F74F223/5F7D14F6/5FACC625" Ref="L?"  Part="1"
 AR Path="/5F74F223/5FACC625" Ref="L?"  Part="1"
-AR Path="/5F74F36B/5F971CD6/5FACC625" Ref="L?"  Part="1"
-F 0 "L?" V 8469 1300 50  0000 C CNN
+AR Path="/5F74F36B/5F971CD6/5FACC625" Ref="L11"  Part="1"
+F 0 "L11" V 8469 1300 50  0000 C CNN
 F 1 "100 uH" V 8560 1300 50  0000 C CNN
 F 2 "Inductor_SMD:L_0603_1608Metric_Pad1.05x0.95mm_HandSolder" H 8650 1300 50  0001 C CNN
@@
 AR Path="/5F74F223/5F7D14F6/5FACC62B" Ref="#PWR?"  Part="1"
 AR Path="/5F74F223/5FACC62B" Ref="#PWR?"  Part="1"
-AR Path="/5F74F36B/5F971CD6/5FACC62B" Ref="#PWR?"  Part="1"
-F 0 "#PWR?" H 9650 1475 50  0001 C CNN
+AR Path="/5F74F36B/5F971CD6/5FACC62B" Ref="#PWR093"  Part="1"
+F 0 "#PWR093" H 9650 1475 50  0001 C CNN
 F 1 "GND" H 9650 1575 50  0000 C CNN
 F 2 "" H 9650 1725 50  0001 C CNN
@@
 AR Path="/5F74F36B/5F821EB2/5FB03A34" Ref="R?"  Part="1"
 AR Path="/5F74F36B/5F8222BE/5FB03A34" Ref="R?"  Part="1"
-AR Path="/5F74F36B/5F971CD6/5FB03A34" Ref="R?"  Part="1"
-F 0 "R?" H 9770 2671 50  0000 L CNN
+AR Path="/5F74F36B/5F971CD6/5FB03A34" Ref="R37"  Part="1"
+F 0 "R37" H 9770 2671 50  0000 L CNN
 F 1 "1.2k" H 9770 2580 50  0000 L CNN
 F 2 "Resistor_SMD:R_0603_1608Metric_Pad0.98x0.95mm_HandSolder" V 9630 2625 50  0001 C CNN
@@
 AR Path="/5F74F36B/5F821EB2/5FB03A3A" Ref="#PWR?"  Part="1"
 AR Path="/5F74F36B/5F8222BE/5FB03A3A" Ref="#PWR?"  Part="1"
-AR Path="/5F74F36B/5F971CD6/5FB03A3A" Ref="#PWR?"  Part="1"
-F 0 "#PWR?" H 9700 2625 50  0001 C CNN
+AR Path="/5F74F36B/5F971CD6/5FB03A3A" Ref="#PWR094"  Part="1"
+F 0 "#PWR094" H 9700 2625 50  0001 C CNN
 F 1 "GND" H 9705 2702 50  0000 C CNN
 F 2 "" H 9700 2875 50  0001 C CNN
@@
 AR Path="/5F74F36B/5F821EB2/5FB03A40" Ref="D?"  Part="1"
 AR Path="/5F74F36B/5F8222BE/5FB03A40" Ref="D?"  Part="1"
-AR Path="/5F74F36B/5F971CD6/5FB03A40" Ref="D?"  Part="1"
-F 0 "D?" V 9739 2108 50  0000 R CNN
+AR Path="/5F74F36B/5F971CD6/5FB03A40" Ref="D24"  Part="1"
+F 0 "D24" V 9739 2108 50  0000 R CNN
 F 1 "Gimbal Logic Green" V 9648 2108 50  0000 R CNN
 F 2 "Diode_SMD:D_0603_1608Metric_Pad1.05x0.95mm_HandSolder" H 9700 2225 50  0001 C CNN

Commit message: Worked on layout
Low current bucks grouped with their componets
Parts:
- C37, C40: footprint Capacitor_THT:CP_Axial_L20.0mm_D10.0mm_P26.00mm_Horizontal -> Capacitor_THT:CP_Radial_D6.3mm_P2.50mm
- C47: footprint Capacitor_THT:CP_Axial_L20.0mm_D10.0mm_P26.00mm_Horizontal -> Capacitor_THT:CP_Radial_D10.0mm_P5.00mm
Other:
- moved on the sheet: D18, D24, R34, R37
Changed lines of the file:
@@
 EESchema Schematic File Version 4
-LIBS:12VBoard_2021_Rev1-cache
 EELAYER 30 0
 EELAYER END
@@
 L Device:R R?
 U 1 1 5F98969B
-P 4300 4150
+P 4300 3750
 AR Path="/5F74F36B/5F821EB2/5F98969B" Ref="R?"  Part="1"
 AR Path="/5F74F36B/5F8222BE/5F98969B" Ref="R?"  Part="1"
 AR Path="/5F74F36B/5F971CD6/5F98969B" Ref="R34"  Part="1"
-F 0 "R34" H 4370 4196 50  0000 L CNN
-F 1 "1.2k" H 4370 4105 50  0000 L CNN
-F 2 "Resistor_SMD:R_0603_1608Metric_Pad0.98x0.95mm_HandSolder" V 4230 4150 50  0001 C CNN
-F 3 "~" H 4300 4150 50  0001 C CNN
-	1    4300 4150
+F 0 "R34" H 4370 3796 50  0000 L CNN
+F 1 "1.2k" H 4370 3705 50  0000 L CNN
+F 2 "Resistor_SMD:R_0603_1608Metric_Pad0.98x0.95mm_HandSolder" V 4230 3750 50  0001 C CNN
+F 3 "~" H 4300 3750 50  0001 C CNN
+	1    4300 3750
 	1    0    0    -1
 $EndComp
@@
 L Device:LED D?
 U 1 1 5F9896A7
-P 4300 3750
+P 4300 4150
 AR Path="/5F74F36B/5F821EB2/5F9896A7" Ref="D?"  Part="1"
 AR Path="/5F74F36B/5F8222BE/5F9896A7" Ref="D?"  Part="1"
 AR Path="/5F74F36B/5F971CD6/5F9896A7" Ref="D18"  Part="1"
-F 0 "D18" V 4339 3633 50  0000 R CNN
-F 1 "Gimbal Acuation Gree" V 4248 3633 50  0000 R CNN
-F 2 "Diode_SMD:D_0603_1608Metric_Pad1.05x0.95mm_HandSolder" H 4300 3750 50  0001 C CNN
-F 3 "~" H 4300 3750 50  0001 C CNN
-	1    4300 3750
+F 0 "D18" V 4339 4033 50  0000 R CNN
+F 1 "Gimbal Acuation Gree" V 4248 4033 50  0000 R CNN
+F 2 "Diode_SMD:D_0603_1608Metric_Pad1.05x0.95mm_HandSolder" H 4300 4150 50  0001 C CNN
+F 3 "~" H 4300 4150 50  0001 C CNN
+	1    4300 4150
 	0    -1   -1   0
 $EndComp
@@
 F 0 "C37" H 2150 3650 50  0000 L CNN
 F 1 "100uF" H 2050 3700 39  0000 L CNN
-F 2 "Capacitor_THT:CP_Axial_L20.0mm_D10.0mm_P26.00mm_Horizontal" H 1950 3700 50  0001 C CNN
+F 2 "Capacitor_THT:CP_Radial_D6.3mm_P2.50mm" H 1950 3700 50  0001 C CNN
 F 3 "~" H 1950 3700 50  0001 C CNN
 	1    1950 3700
@@
 F 0 "C40" H 2550 3650 50  0000 L CNN
 F 1 "100uF" H 2450 3700 39  0000 L CNN
-F 2 "Capacitor_THT:CP_Axial_L20.0mm_D10.0mm_P26.00mm_Horizontal" H 2350 3700 50  0001 C CNN
+F 2 "Capacitor_THT:CP_Radial_D6.3mm_P2.50mm" H 2350 3700 50  0001 C CNN
 F 3 "~" H 2350 3700 50  0001 C CNN
 	1    2350 3700
@@
 F 0 "C47" V 8875 1475 50  0000 L CNN
 F 1 "1000 uF" V 8950 1400 50  0000 L CNN
-F 2 "Capacitor_THT:CP_Axial_L20.0mm_D10.0mm_P26.00mm_Horizontal" H 9100 1525 50  0001 C CNN
+F 2 "Capacitor_THT:CP_Radial_D10.0mm_P5.00mm" H 9100 1525 50  0001 C CNN
 F 3 "~" H 9100 1525 50  0001 C CNN
 	1    9100 1525
@@
 L Device:R R?
 U 1 1 5FB03A34
-P 9700 2625
+P 9700 2225
 AR Path="/5F74F36B/5F821EB2/5FB03A34" Ref="R?"  Part="1"
 AR Path="/5F74F36B/5F8222BE/5FB03A34" Ref="R?"  Part="1"
 AR Path="/5F74F36B/5F971CD6/5FB03A34" Ref="R37"  Part="1"
-F 0 "R37" H 9770 2671 50  0000 L CNN
-F 1 "1.2k" H 9770 2580 50  0000 L CNN
-F 2 "Resistor_SMD:R_0603_1608Metric_Pad0.98x0.95mm_HandSolder" V 9630 2625 50  0001 C CNN
-F 3 "~" H 9700 2625 50  0001 C CNN
-	1    9700 2625
+F 0 "R37" H 9770 2271 50  0000 L CNN
+F 1 "1.2k" H 9770 2180 50  0000 L CNN
+F 2 "Resistor_SMD:R_0603_1608Metric_Pad0.98x0.95mm_HandSolder" V 9630 2225 50  0001 C CNN
+F 3 "~" H 9700 2225 50  0001 C CNN
+	1    9700 2225
 	1    0    0    -1
 $EndComp
@@
 L Device:LED D?
 U 1 1 5FB03A40
-P 9700 2225
+P 9700 2625
 AR Path="/5F74F36B/5F821EB2/5FB03A40" Ref="D?"  Part="1"
 AR Path="/5F74F36B/5F8222BE/5FB03A40" Ref="D?"  Part="1"
 AR Path="/5F74F36B/5F971CD6/5FB03A40" Ref="D24"  Part="1"
-F 0 "D24" V 9739 2108 50  0000 R CNN
-F 1 "Gimbal Logic Green" V 9648 2108 50  0000 R CNN
-F 2 "Diode_SMD:D_0603_1608Metric_Pad1.05x0.95mm_HandSolder" H 9700 2225 50  0001 C CNN
-F 3 "~" H 9700 2225 50  0001 C CNN
-	1    9700 2225
+F 0 "D24" V 9739 2508 50  0000 R CNN
+F 1 "Gimbal Logic Green" V 9648 2508 50  0000 R CNN
+F 2 "Diode_SMD:D_0603_1608Metric_Pad1.05x0.95mm_HandSolder" H 9700 2625 50  0001 C CNN
+F 3 "~" H 9700 2625 50  0001 C CNN
+	1    9700 2625
 	0    -1   -1   0
 $EndComp

Commit message: Fixed Resistor and Capasitor footprints
found other issues
Parts:
- C33, C34, C35, C36, C38, C39, C41, C42: footprint Capacitor_SMD:C_0603_1608Metric_Pad1.08x0.95mm_HandSolder -> Capacitor_SMD:C_0603_1608Metric_Pad1.05x0.95mm_HandSolder
- R27, R28, R29, R30, R31, R32, R34, R37: footprint Resistor_SMD:R_0603_1608Metric_Pad0.98x0.95mm_HandSolder -> Resistor_SMD:R_0603_1608Metric_Pad1.05x0.95mm_HandSolder
Changed lines of the file:
@@
 F 0 "R34" H 4370 3796 50  0000 L CNN
 F 1 "1.2k" H 4370 3705 50  0000 L CNN
-F 2 "Resistor_SMD:R_0603_1608Metric_Pad0.98x0.95mm_HandSolder" V 4230 3750 50  0001 C CNN
+F 2 "Resistor_SMD:R_0603_1608Metric_Pad1.05x0.95mm_HandSolder" V 4230 3750 50  0001 C CNN
 F 3 "~" H 4300 3750 50  0001 C CNN
 	1    4300 3750
@@
 F 0 "R31" H 1859 4646 50  0000 L CNN
 F 1 "9.76k" H 1859 4555 50  0000 L CNN
-F 2 "Resistor_SMD:R_0603_1608Metric_Pad0.98x0.95mm_HandSolder" H 1800 4600 50  0001 C CNN
+F 2 "Resistor_SMD:R_0603_1608Metric_Pad1.05x0.95mm_HandSolder" H 1800 4600 50  0001 C CNN
 F 3 "~" H 1800 4600 50  0001 C CNN
 	1    1800 4600
@@
 F 0 "R32" H 2409 2196 50  0000 L CNN
 F 1 "261K" H 2409 2105 50  0000 L CNN
-F 2 "Resistor_SMD:R_0603_1608Metric_Pad0.98x0.95mm_HandSolder" H 2350 2150 50  0001 C CNN
+F 2 "Resistor_SMD:R_0603_1608Metric_Pad1.05x0.95mm_HandSolder" H 2350 2150 50  0001 C CNN
 F 3 "~" H 2350 2150 50  0001 C CNN
 	1    2350 2150
@@
 F 0 "R28" H 1609 996 50  0000 L CNN
 F 1 "36.5K" H 1609 905 50  0000 L CNN
-F 2 "Resistor_SMD:R_0603_1608Metric_Pad0.98x0.95mm_HandSolder" H 1550 950 50  0001 C CNN
+F 2 "Resistor_SMD:R_0603_1608Metric_Pad1.05x0.95mm_HandSolder" H 1550 950 50  0001 C CNN
 F 3 "~" H 1550 950 50  0001 C CNN
 	1    1550 950
@@
 F 0 "R29" H 1609 1296 50  0000 L CNN
 F 1 "2.26K" H 1609 1205 50  0000 L CNN
-F 2 "Resistor_SMD:R_0603_1608Metric_Pad0.98x0.95mm_HandSolder" H 1550 1250 50  0001 C CNN
+F 2 "Resistor_SMD:R_0603_1608Metric_Pad1.05x0.95mm_HandSolder" H 1550 1250 50  0001 C CNN
 F 3 "~" H 1550 1250 50  0001 C CNN
 	1    1550 1250
@@
 F 0 "R30" H 1859 4346 50  0000 L CNN
 F 1 "86.6K" H 1859 4255 50  0000 L CNN
-F 2 "Resistor_SMD:R_0603_1608Metric_Pad0.98x0.95mm_HandSolder" H 1800 4300 50  0001 C CNN
+F 2 "Resistor_SMD:R_0603_1608Metric_Pad1.05x0.95mm_HandSolder" H 1800 4300 50  0001 C CNN
 F 3 "~" H 1800 4300 50  0001 C CNN
 	1    1800 4300
@@
 F 0 "R27" H 1359 4246 50  0000 L CNN
 F 1 "5m" H 1359 4155 50  0000 L CNN
-F 2 "Resistor_SMD:R_0603_1608Metric_Pad0.98x0.95mm_HandSolder" H 1300 4200 50  0001 C CNN
+F 2 "Resistor_SMD:R_0603_1608Metric_Pad1.05x0.95mm_HandSolder" H 1300 4200 50  0001 C CNN
 F 3 "~" H 1300 4200 50  0001 C CNN
 	1    1300 4200
@@
 F 0 "C34" H 1242 1046 50  0000 L CNN
 F 1 "2.2uF" H 1242 955 50  0000 L CNN
-F 2 "Capacitor_SMD:C_0603_1608Metric_Pad1.08x0.95mm_HandSolder" H 1150 1000 50  0001 C CNN
+F 2 "Capacitor_SMD:C_0603_1608Metric_Pad1.05x0.95mm_HandSolder" H 1150 1000 50  0001 C CNN
 F 3 "~" H 1150 1000 50  0001 C CNN
 	1    1150 1000
@@
 F 0 "C36" H 1442 1046 50  0000 L CNN
 F 1 "100nF" H 1442 955 50  0000 L CNN
-F 2 "Capacitor_SMD:C_0603_1608Metric_Pad1.08x0.95mm_HandSolder" H 1350 1000 50  0001 C CNN
+F 2 "Capacitor_SMD:C_0603_1608Metric_Pad1.05x0.95mm_HandSolder" H 1350 1000 50  0001 C CNN
 F 3 "~" H 1350 1000 50  0001 C CNN
 	1    1350 1000
@@
 F 0 "C41" V 2271 1200 50  0000 C CNN
 F 1 "470pF" V 2362 1200 50  0000 C CNN
-F 2 "Capacitor_SMD:C_0603_1608Metric_Pad1.08x0.95mm_HandSolder" H 2500 1200 50  0001 C CNN
+F 2 "Capacitor_SMD:C_0603_1608Metric_Pad1.05x0.95mm_HandSolder" H 2500 1200 50  0001 C CNN
 F 3 "~" H 2500 1200 50  0001 C CNN
 	1    2500 1200
@@
 F 0 "C42" V 2271 1400 50  0000 C CNN
 F 1 "33nF" V 2362 1400 50  0000 C CNN
-F 2 "Capacitor_SMD:C_0603_1608Metric_Pad1.08x0.95mm_HandSolder" H 2500 1400 50  0001 C CNN
+F 2 "Capacitor_SMD:C_0603_1608Metric_Pad1.05x0.95mm_HandSolder" H 2500 1400 50  0001 C CNN
 F 3 "~" H 2500 1400 50  0001 C CNN
 	1    2500 1400
@@
 F 0 "C38" H 2292 1946 50  0000 L CNN
 F 1 "10pF" H 2292 1855 50  0000 L CNN
-F 2 "Capacitor_SMD:C_0603_1608Metric_Pad1.08x0.95mm_HandSolder" H 2200 1900 50  0001 C CNN
+F 2 "Capacitor_SMD:C_0603_1608Metric_Pad1.05x0.95mm_HandSolder" H 2200 1900 50  0001 C CNN
 F 3 "~" H 2200 1900 50  0001 C CNN
 	1    2200 1900
@@
 F 0 "C39" H 2442 1946 50  0000 L CNN
 F 1 "120pF" H 2442 1855 50  0000 L CNN
-F 2 "Capacitor_SMD:C_0603_1608Metric_Pad1.08x0.95mm_HandSolder" H 2350 1900 50  0001 C CNN
+F 2 "Capacitor_SMD:C_0603_1608Metric_Pad1.05x0.95mm_HandSolder" H 2350 1900 50  0001 C CNN
 F 3 "~" H 2350 1900 50  0001 C CNN
 	1    2350 1900
@@
 F 0 "C35" H 1292 2696 50  0000 L CNN
 F 1 "1uF" H 1292 2605 50  0000 L CNN
-F 2 "Capacitor_SMD:C_0603_1608Metric_Pad1.08x0.95mm_HandSolder" H 1200 2650 50  0001 C CNN
+F 2 "Capacitor_SMD:C_0603_1608Metric_Pad1.05x0.95mm_HandSolder" H 1200 2650 50  0001 C CNN
 F 3 "~" H 1200 2650 50  0001 C CNN
 	1    1200 2650
@@
 F 0 "C33" H 1142 2996 50  0000 L CNN
 F 1 "100nF" H 1142 2905 50  0000 L CNN
-F 2 "Capacitor_SMD:C_0603_1608Metric_Pad1.08x0.95mm_HandSolder" H 1050 2950 50  0001 C CNN
+F 2 "Capacitor_SMD:C_0603_1608Metric_Pad1.05x0.95mm_HandSolder" H 1050 2950 50  0001 C CNN
 F 3 "~" H 1050 2950 50  0001 C CNN
 	1    1050 2950
@@
 F 0 "R37" H 9770 2271 50  0000 L CNN
 F 1 "1.2k" H 9770 2180 50  0000 L CNN
-F 2 "Resistor_SMD:R_0603_1608Metric_Pad0.98x0.95mm_HandSolder" V 9630 2225 50  0001 C CNN
+F 2 "Resistor_SMD:R_0603_1608Metric_Pad1.05x0.95mm_HandSolder" V 9630 2225 50  0001 C CNN
 F 3 "~" H 9700 2225 50  0001 C CNN
 	1    9700 2225

Commit message: Components
Added the correct mosfets for the extra and the high current bucks
Parts:
- removed Q6, Q7: 2N7000, Package_TO_SOT_THT:TO-92_Inline, symbol Transistor_FET:2N7000
- added Q6: CSD18537NQ5A, symbol 12VBoard_2021_Rev1-rescue:CSD18537NQ5A
- added Q7: CSD18531Q5A, symbol 12VBoard_2021_Rev1-rescue:CSD18531Q5A
Connections:
- wire segments 150 -> 174
Other:
- moved on the sheet: R27
Changed lines of the file:
@@
 L power:GND #PWR068
 U 1 1 5FB8B439
-P 1300 4400
-F 0 "#PWR068" H 1300 4150 50  0001 C CNN
-F 1 "GND" H 1305 4227 50  0000 C CNN
-F 2 "" H 1300 4400 50  0001 C CNN
-F 3 "" H 1300 4400 50  0001 C CNN
-	1    1300 4400
+P 1300 4800
+F 0 "#PWR068" H 1300 4550 50  0001 C CNN
+F 1 "GND" H 1305 4627 50  0000 C CNN
+F 2 "" H 1300 4800 50  0001 C CNN
+F 3 "" H 1300 4800 50  0001 C CNN
+	1    1300 4800
 	1    0    0    -1
 $EndComp
@@
 Wire Wire Line
 	1200 2750 1200 2800
-Text HLabel 1350 3050 2    50   Input ~ 0
+Text HLabel 1875 2850 2    50   Input ~ 0
 PackVoltage
-$Comp
-L Transistor_FET:2N7000 Q6
-U 1 1 5FB3AE97
-P 1150 3300
-F 0 "Q6" H 1354 3346 50  0000 L CNN
-F 1 "2N7000" H 1354 3255 50  0000 L CNN
-F 2 "Package_TO_SOT_THT:TO-92_Inline" H 1350 3225 50  0001 L CIN
-F 3 "https://www.fairchildsemi.com/datasheets/2N/2N7000.pdf" H 1150 3300 50  0001 L CNN
-	1    1150 3300
-	1    0    0    -1
-$EndComp
-Wire Wire Line
-	1350 3050 1250 3050
-Wire Wire Line
-	1250 3050 1250 3100
-$Comp
-L Transistor_FET:2N7000 Q7
-U 1 1 5FB57A80
-P 1200 3800
-F 0 "Q7" H 1404 3846 50  0000 L CNN
-F 1 "2N7000" H 1404 3755 50  0000 L CNN
-F 2 "Package_TO_SOT_THT:TO-92_Inline" H 1400 3725 50  0001 L CIN
-F 3 "https://www.fairchildsemi.com/datasheets/2N/2N7000.pdf" H 1200 3800 50  0001 L CNN
-	1    1200 3800
-	1    0    0    -1
-$EndComp
-Wire Wire Line
-	1250 3500 1250 3550
 Wire Wire Line
 	1250 3550 1300 3550
-Wire Wire Line
-	1300 3550 1300 3600
 Wire Wire Line
 	1050 3050 1050 3550
@@
 L Device:R_Small R27
 U 1 1 5FB854FB
-P 1300 4200
-F 0 "R27" H 1359 4246 50  0000 L CNN
-F 1 "5m" H 1359 4155 50  0000 L CNN
-F 2 "Resistor_SMD:R_0603_1608Metric_Pad1.05x0.95mm_HandSolder" H 1300 4200 50  0001 C CNN
-F 3 "~" H 1300 4200 50  0001 C CNN
-	1    1300 4200
-	1    0    0    -1
-$EndComp
-Wire Wire Line
-	1300 4000 1300 4050
-Wire Wire Line
-	1300 4300 1300 4350
-Text GLabel 900  3300 0    50   Input ~ 0
+P 1300 4600
+F 0 "R27" H 1359 4646 50  0000 L CNN
+F 1 "5m" H 1359 4555 50  0000 L CNN
+F 2 "Resistor_SMD:R_0603_1608Metric_Pad1.05x0.95mm_HandSolder" H 1300 4600 50  0001 C CNN
+F 3 "~" H 1300 4600 50  0001 C CNN
+	1    1300 4600
+	1    0    0    -1
+$EndComp
+Wire Wire Line
+	1300 4700 1300 4750
+Text GLabel 1825 3350 3    50   Input ~ 0
 HO
-Text GLabel 950  3800 0    50   Input ~ 0
+Text GLabel 1600 4150 3    50   Input ~ 0
 LO
-Wire Wire Line
-	950  3300 900  3300
-Wire Wire Line
-	1000 3800 950  3800
 Wire Wire Line
 	1050 2750 1050 2800
@@
 Wire Wire Line
 	1050 2550 1050 2500
-Text GLabel 1250 4050 0    50   Input ~ 0
+Text GLabel 1250 4450 0    50   Input ~ 0
 CS
-Text GLabel 1250 4350 0    50   Input ~ 0
+Text GLabel 1250 4750 0    50   Input ~ 0
 CSGDEMB
 Wire Wire Line
-	1300 4050 1250 4050
-Connection ~ 1300 4050
-Wire Wire Line
-	1300 4050 1300 4100
-Wire Wire Line
-	1300 4350 1250 4350
-Connection ~ 1300 4350
-Wire Wire Line
-	1300 4350 1300 4400
+	1300 4450 1250 4450
+Connection ~ 1300 4450
+Wire Wire Line
+	1300 4450 1300 4500
+Wire Wire Line
+	1300 4750 1250 4750
+Connection ~ 1300 4750
+Wire Wire Line
+	1300 4750 1300 4800
 $Comp
 L Device:CP1_Small C37
@@
 Text HLabel 6450 1300 0    49   Input ~ 0
 CTL_Gimbal
+$Comp
+L 12VBoard_2021_Rev1-rescue:CSD18537NQ5A Q?
+U 1 1 5FD3AF2E
+P 1675 3100
+AR Path="/5F74F36B/5F8236F9/5FD3AF2E" Ref="Q?"  Part="1"
+AR Path="/5F74F36B/5F971CD6/5FD3AF2E" Ref="Q6"  Part="1"
+F 0 "Q6" V 1600 2875 50  0000 R CNN
+F 1 "CSD18537NQ5A" V 1725 2900 50  0000 R CNN
+F 2 "" H 1675 3100 50  0001 C CNN
+F 3 "" H 1675 3100 50  0001 C CNN
+	1    1675 3100
+	0    -1   -1   0
+$EndComp
+$Comp
+L 12VBoard_2021_Rev1-rescue:CSD18531Q5A Q?
+U 1 1 5FD3AF34
+P 1450 3900
+AR Path="/5F74F36B/5F8236F9/5FD3AF34" Ref="Q?"  Part="1"
+AR Path="/5F74F36B/5F971CD6/5FD3AF34" Ref="Q7"  Part="1"
+F 0 "Q7" V 1400 4225 50  0000 R CNN
+F 1 "CSD18531Q5A" V 1475 4650 50  0000 R CNN
+F 2 "" H 1450 3950 50  0001 C CNN
+F 3 "" H 1450 3950 50  0001 C CNN
+	1    1450 3900
+	0    -1   -1   0
+$EndComp
+Wire Wire Line
+	1600 4150 1600 4100
+Wire Wire Line
+	1500 4100 1500 4150
+Wire Wire Line
+	1500 4150 1400 4150
+Wire Wire Line
+	1300 4150 1300 4100
+Wire Wire Line
+	1300 4150 1300 4450
+Connection ~ 1300 4150
+Wire Wire Line
+	1400 4100 1400 4150
+Connection ~ 1400 4150
+Wire Wire Line
+	1400 4150 1300 4150
+Wire Wire Line
+	1600 3700 1600 3650
+Wire Wire Line
+	1600 3650 1500 3650
+Wire Wire Line
+	1300 3550 1300 3650
+Wire Wire Line
+	1300 3650 1300 3700
+Connection ~ 1300 3650
+Wire Wire Line
+	1400 3700 1400 3650
+Connection ~ 1400 3650
+Wire Wire Line
+	1400 3650 1300 3650
+Wire Wire Line
+	1500 3700 1500 3650
+Connection ~ 1500 3650
+Wire Wire Line
+	1500 3650 1400 3650
+Wire Wire Line
+	1875 2850 1825 2850
+Wire Wire Line
+	1525 2850 1525 2900
+Wire Wire Line
+	1625 2900 1625 2850
+Connection ~ 1625 2850
+Wire Wire Line
+	1625 2850 1525 2850
+Wire Wire Line
+	1725 2900 1725 2850
+Connection ~ 1725 2850
+Wire Wire Line
+	1725 2850 1625 2850
+Wire Wire Line
+	1825 2900 1825 2850
+Connection ~ 1825 2850
+Wire Wire Line
+	1825 2850 1725 2850
+Wire Wire Line
+	1825 3350 1825 3300
+Wire Wire Line
+	1250 3350 1525 3350
+Wire Wire Line
+	1725 3350 1725 3300
+Wire Wire Line
+	1250 3350 1250 3550
+Wire Wire Line
+	1625 3300 1625 3350
+Connection ~ 1625 3350
+Wire Wire Line
+	1625 3350 1725 3350
+Wire Wire Line
+	1525 3300 1525 3350
+Connection ~ 1525 3350
+Wire Wire Line
+	1525 3350 1625 3350
 $EndSCHEMATC
