File: Hardware/12VBoard_2021_Rev1/Gimbal.sch (KiCad schematic (older format))
At the start: 35 parts, among them Q6 CSD18537NQ5A, Q7 CSD18531Q5A, U12 LM5116, U13 INA198, U16 LM2576S-12/NOPB

Commit message: updated footprints
Parts:
- D23: footprint Diode_SMD:D_0603_1608Metric_Pad1.05x0.95mm_HandSolder -> Diode_THT:D_DO-201AD_P15.24mm_Horizontal
- Q6, Q7: footprint (none) -> Package_SON:VSONP-8-1EP_5x6_P1.27mm
Changed lines of the file:
@@
 F 0 "D23" V 8254 1605 50  0000 L CNN
 F 1 "D_Schottky" V 8345 1605 50  0000 L CNN
-F 2 "Diode_SMD:D_0603_1608Metric_Pad1.05x0.95mm_HandSolder" H 8300 1525 50  0001 C CNN
+F 2 "Diode_THT:D_DO-201AD_P15.24mm_Horizontal" H 8300 1525 50  0001 C CNN
 F 3 "~" H 8300 1525 50  0001 C CNN
 	1    8300 1525
@@
 F 0 "Q6" V 1600 2875 50  0000 R CNN
 F 1 "CSD18537NQ5A" V 1725 2900 50  0000 R CNN
-F 2 "" H 1675 3100 50  0001 C CNN
+F 2 "Package_SON:VSONP-8-1EP_5x6_P1.27mm" H 1675 3100 50  0001 C CNN
 F 3 "" H 1675 3100 50  0001 C CNN
 	1    1675 3100
@@
 F 0 "Q7" V 1400 4225 50  0000 R CNN
 F 1 "CSD18531Q5A" V 1475 4650 50  0000 R CNN
-F 2 "" H 1450 3950 50  0001 C CNN
+F 2 "Package_SON:VSONP-8-1EP_5x6_P1.27mm" H 1450 3950 50  0001 C CNN
 F 3 "" H 1450 3950 50  0001 C CNN
 	1    1450 3900
