File: Hardware/12VBoard_2021_Rev1/_autosave-12VBoard_2021_Rev1.kicad_pcb (KiCad board)
At the start: 2 copper layers, 101.6 x 129.4 mm, 135 parts, among them Q10 IRLML2060, Q11 IRLML2060, Q12 IRLML2060, Q13 IRLML2060, Q3 IRLML2060, Q8 IRLML2060, Q9 IRLML2060, U1 LT1910, U10 INA198, U11 FDS66900AS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

Commit message: admin changes
-current sensing on high current
-fixed traces for current sensing
Routing:
- net /High Current Outputs/12VActuation: track 25.1 -> 29.5 mm, vias 3 -> 0
- net Net-(F1-Pad2): track 5.81 -> 8.68 mm, vias 0 -> 1
- net Net-(F4-Pad2): track 6.16 -> 5.33 mm, vias 0 -> 1
- net Net-(F3-Pad2): track 5.78 -> 4.96 mm, vias 0 -> 1
- net GND: vias 5 -> 27
