File: Hardware/2022_Rev2/BuckAndersons.sch (KiCad schematic (older format))
At the start: 27 parts

Commit message: Added Heirarchical Labels inside the 12V sheet
Parts:
- Conn? (x15): symbol MRDT_Connectors:AndersonPP -> 2022_Rev2-rescue:AndersonPP-MRDT_Connectors
Changed lines of the file:
@@
 $EndDescr
 $Comp
-L MRDT_Connectors:AndersonPP Conn?
+L 2022_Rev2-rescue:AndersonPP-MRDT_Connectors Conn?
 U 4 1 621C7125
 P 4700 1400
+AR Path="/621C7125" Ref="Conn?"  Part="4"
+AR Path="/6217B740/621C7125" Ref="Conn?"  Part="4"
 F 0 "Conn?" H 4908 1787 60  0000 C CNN
 F 1 "Aux_1_Out" H 4908 1681 60  0000 C CNN
@@
 $EndComp
 $Comp
-L MRDT_Connectors:AndersonPP Conn?
+L 2022_Rev2-rescue:AndersonPP-MRDT_Connectors Conn?
 U 2 1 621C7C59
 P 4700 1900
+AR Path="/621C7C59" Ref="Conn?"  Part="2"
+AR Path="/6217B740/621C7C59" Ref="Conn?"  Part="2"
 F 0 "Conn?" H 4908 2287 60  0000 C CNN
 F 1 "Aux_1_Out" H 4908 2181 60  0000 C CNN
@@
 $EndComp
 $Comp
-L MRDT_Connectors:AndersonPP Conn?
+L 2022_Rev2-rescue:AndersonPP-MRDT_Connectors Conn?
 U 1 1 621C871C
 P 4700 2400
+AR Path="/621C871C" Ref="Conn?"  Part="1"
+AR Path="/6217B740/621C871C" Ref="Conn?"  Part="1"
 F 0 "Conn?" H 4908 2787 60  0000 C CNN
 F 1 "Aux_1_Out" H 4908 2681 60  0000 C CNN
@@
 Aux_1_Toggle
 $Comp
-L MRDT_Connectors:AndersonPP Conn?
+L 2022_Rev2-rescue:AndersonPP-MRDT_Connectors Conn?
 U 4 1 621CF26B
 P 4700 3500
+AR Path="/621CF26B" Ref="Conn?"  Part="4"
+AR Path="/6217B740/621CF26B" Ref="Conn?"  Part="4"
 F 0 "Conn?" H 4908 3887 60  0000 C CNN
 F 1 "Aux_2_Out" H 4908 3781 60  0000 C CNN
@@
 $EndComp
 $Comp
-L MRDT_Connectors:AndersonPP Conn?
+L 2022_Rev2-rescue:AndersonPP-MRDT_Connectors Conn?
 U 2 1 621CF271
 P 4700 4000
+AR Path="/621CF271" Ref="Conn?"  Part="2"
+AR Path="/6217B740/621CF271" Ref="Conn?"  Part="2"
 F 0 "Conn?" H 4908 4387 60  0000 C CNN
 F 1 "Aux_2_Out" H 4908 4281 60  0000 C CNN
@@
 $EndComp
 $Comp
-L MRDT_Connectors:AndersonPP Conn?
+L 2022_Rev2-rescue:AndersonPP-MRDT_Connectors Conn?
 U 1 1 621CF277
 P 4700 4500
+AR Path="/621CF277" Ref="Conn?"  Part="1"
+AR Path="/6217B740/621CF277" Ref="Conn?"  Part="1"
 F 0 "Conn?" H 4908 4887 60  0000 C CNN
 F 1 "Aux_2_Out" H 4908 4781 60  0000 C CNN
@@
 Aux_2_Toggle
 $Comp
-L MRDT_Connectors:AndersonPP Conn?
+L 2022_Rev2-rescue:AndersonPP-MRDT_Connectors Conn?
 U 3 1 62262695
 P 6200 1400
+AR Path="/62262695" Ref="Conn?"  Part="3"
+AR Path="/6217B740/62262695" Ref="Conn?"  Part="3"
 F 0 "Conn?" H 6408 1787 60  0000 C CNN
 F 1 "Aux_1_In" H 6408 1681 60  0000 C CNN
@@
 $EndComp
 $Comp
-L MRDT_Connectors:AndersonPP Conn?
+L 2022_Rev2-rescue:AndersonPP-MRDT_Connectors Conn?
 U 1 1 62264AAC
 P 6200 1900
+AR Path="/62264AAC" Ref="Conn?"  Part="1"
+AR Path="/6217B740/62264AAC" Ref="Conn?"  Part="1"
 F 0 "Conn?" H 6408 2287 60  0000 C CNN
 F 1 "Aux_1_In" H 6408 2181 60  0000 C CNN
@@
 	6600 1300 6800 1300
 $Comp
-L MRDT_Connectors:AndersonPP Conn?
+L 2022_Rev2-rescue:AndersonPP-MRDT_Connectors Conn?
 U 3 1 62267828
 P 6200 3500
+AR Path="/62267828" Ref="Conn?"  Part="3"
+AR Path="/6217B740/62267828" Ref="Conn?"  Part="3"
 F 0 "Conn?" H 6408 3887 60  0000 C CNN
 F 1 "Aux_2_In" H 6408 3781 60  0000 C CNN
@@
 $EndComp
 $Comp
-L MRDT_Connectors:AndersonPP Conn?
+L 2022_Rev2-rescue:AndersonPP-MRDT_Connectors Conn?
 U 1 1 6226782E
 P 6200 4000
+AR Path="/6226782E" Ref="Conn?"  Part="1"
+AR Path="/6217B740/6226782E" Ref="Conn?"  Part="1"
 F 0 "Conn?" H 6408 4387 60  0000 C CNN
 F 1 "Aux_2_In" H 6408 4281 60  0000 C CNN
@@
 	6600 3400 6800 3400
 $Comp
-L MRDT_Connectors:AndersonPP Conn?
+L 2022_Rev2-rescue:AndersonPP-MRDT_Connectors Conn?
 U 4 1 6226B6C1
 P 1400 5650
+AR Path="/6226B6C1" Ref="Conn?"  Part="4"
+AR Path="/6217B740/6226B6C1" Ref="Conn?"  Part="4"
 F 0 "Conn?" H 1608 6037 60  0000 C CNN
 F 1 "Aux_GP_Out" H 1608 5931 60  0000 C CNN
@@
 $EndComp
 $Comp
-L MRDT_Connectors:AndersonPP Conn?
+L 2022_Rev2-rescue:AndersonPP-MRDT_Connectors Conn?
 U 2 1 6226B6C7
 P 1400 6150
+AR Path="/6226B6C7" Ref="Conn?"  Part="2"
+AR Path="/6217B740/6226B6C7" Ref="Conn?"  Part="2"
 F 0 "Conn?" H 1608 6537 60  0000 C CNN
 F 1 "Aux_GP_Out" H 1608 6431 60  0000 C CNN
@@
 $EndComp
 $Comp
-L MRDT_Connectors:AndersonPP Conn?
+L 2022_Rev2-rescue:AndersonPP-MRDT_Connectors Conn?
 U 1 1 6226B6CD
 P 1400 6650
+AR Path="/6226B6CD" Ref="Conn?"  Part="1"
+AR Path="/6217B740/6226B6CD" Ref="Conn?"  Part="1"
 F 0 "Conn?" H 1608 7037 60  0000 C CNN
 F 1 "Aux_GP_Out" H 1608 6931 60  0000 C CNN
@@
 GP_Toggle
 $Comp
-L MRDT_Connectors:AndersonPP Conn?
+L 2022_Rev2-rescue:AndersonPP-MRDT_Connectors Conn?
 U 3 1 6226B6DF
 P 2900 5650
+AR Path="/6226B6DF" Ref="Conn?"  Part="3"
+AR Path="/6217B740/6226B6DF" Ref="Conn?"  Part="3"
 F 0 "Conn?" H 3108 6037 60  0000 C CNN
 F 1 "Aux_GP_In" H 3108 5931 60  0000 C CNN
@@
 $EndComp
 $Comp
-L MRDT_Connectors:AndersonPP Conn?
+L 2022_Rev2-rescue:AndersonPP-MRDT_Connectors Conn?
 U 1 1 6226B6E5
 P 2900 6150
+AR Path="/6226B6E5" Ref="Conn?"  Part="1"
+AR Path="/6217B740/6226B6E5" Ref="Conn?"  Part="1"
 F 0 "Conn?" H 3108 6537 60  0000 C CNN
 F 1 "Aux_GP_In" H 3108 6431 60  0000 C CNN

Commit message: assigning footprints pt.1
Parts:
- C10, C9: renamed from C?; footprint (none) -> Capacitor_SMD:C_0603_1608Metric_Pad1.08x0.95mm_HandSolder
- C11, C12, C7, C8: renamed from C?; footprint (none) -> Capacitor_THT:CP_Radial_D6.3mm_P2.50mm
- D3, D4: renamed from D?; footprint (none) -> Diode_SMD:D_0603_1608Metric_Pad1.05x0.95mm_HandSolder
- gave numbers to parts that had none: 10
