File: Hardware/2022_Rev2/2022_Rev2.sch (KiCad schematic (older format))
At the start: 24 parts, among them U1 OKI-78SR-5_1.5-W36-C, U2 OKI-78SR-3.3_1.5-W36-C

Commit message: fixed footprints
Parts:
- Conn10, Conn11, Conn12, Conn4, Conn5, Conn6, Conn7, Conn8: footprint MRDT_Connectors:Anderson_2_Horizontal_Side_by_Side_PV -> MRDT_Connectors:Anderson_2_Vertical_Sidy_by_Side
- Conn9: footprint MRDT_Connectors:Anderson_3_Horizontal_Side_by_Side -> MRDT_Connectors:Anderson_3_Vertical_Side_by_Side
Changed lines of the file:
@@
 F 0 "Conn4" V 9450 750 60  0000 C CNN
 F 1 "AndersonPP" V 9350 750 60  0000 C CNN
-F 2 "MRDT_Connectors:Anderson_2_Horizontal_Side_by_Side_PV" H 9350 100 60  0001 C CNN
+F 2 "MRDT_Connectors:Anderson_2_Vertical_Sidy_by_Side" H 9350 100 60  0001 C CNN
 F 3 "" H 9350 100 60  0001 C CNN
 	2    9500 650
@@
 F 0 "Conn9" V 10550 3750 60  0000 C CNN
 F 1 "AndersonPP" V 10450 3750 60  0000 C CNN
-F 2 "MRDT_Connectors:Anderson_3_Horizontal_Side_by_Side" H 10450 3100 60  0001 C CNN
+F 2 "MRDT_Connectors:Anderson_3_Vertical_Side_by_Side" H 10450 3100 60  0001 C CNN
 F 3 "" H 10450 3100 60  0001 C CNN
 	1    10600 3650
@@
 F 0 "Conn4" V 10000 750 60  0000 C CNN
 F 1 "AndersonPP" V 9900 750 60  0000 C CNN
-F 2 "MRDT_Connectors:Anderson_2_Horizontal_Side_by_Side_PV" H 9900 100 60  0001 C CNN
+F 2 "MRDT_Connectors:Anderson_2_Vertical_Sidy_by_Side" H 9900 100 60  0001 C CNN
 F 3 "" H 9900 100 60  0001 C CNN
 	1    10050 650
@@
 F 0 "Conn5" V 10000 1350 60  0000 C CNN
 F 1 "AndersonPP" V 9900 1350 60  0000 C CNN
-F 2 "MRDT_Connectors:Anderson_2_Horizontal_Side_by_Side_PV" H 9900 700 60  0001 C CNN
+F 2 "MRDT_Connectors:Anderson_2_Vertical_Sidy_by_Side" H 9900 700 60  0001 C CNN
 F 3 "" H 9900 700 60  0001 C CNN
 	1    10050 1250
@@
 F 0 "Conn6" V 10000 1950 60  0000 C CNN
 F 1 "AndersonPP" V 9900 1950 60  0000 C CNN
-F 2 "MRDT_Connectors:Anderson_2_Horizontal_Side_by_Side_PV" H 9900 1300 60  0001 C CNN
+F 2 "MRDT_Connectors:Anderson_2_Vertical_Sidy_by_Side" H 9900 1300 60  0001 C CNN
 F 3 "" H 9900 1300 60  0001 C CNN
 	1    10050 1850
@@
 F 0 "Conn7" V 10000 2550 60  0000 C CNN
 F 1 "AndersonPP" V 9900 2550 60  0000 C CNN
-F 2 "MRDT_Connectors:Anderson_2_Horizontal_Side_by_Side_PV" H 9900 1900 60  0001 C CNN
+F 2 "MRDT_Connectors:Anderson_2_Vertical_Sidy_by_Side" H 9900 1900 60  0001 C CNN
 F 3 "" H 9900 1900 60  0001 C CNN
 	1    10050 2450
@@
 F 0 "Conn9" H 9800 4150 60  0000 C CNN
 F 1 "AndersonPP" V 9600 4000 60  0000 C CNN
-F 2 "MRDT_Connectors:Anderson_3_Horizontal_Side_by_Side" H 9550 3350 60  0001 C CNN
+F 2 "MRDT_Connectors:Anderson_3_Vertical_Side_by_Side" H 9550 3350 60  0001 C CNN
 F 3 "" H 9550 3350 60  0001 C CNN
 	3    9700 3900
@@
 F 0 "Conn10" V 10000 4350 60  0000 C CNN
 F 1 "AndersonPP" V 9900 4350 60  0000 C CNN
-F 2 "MRDT_Connectors:Anderson_2_Horizontal_Side_by_Side_PV" H 9900 3700 60  0001 C CNN
+F 2 "MRDT_Connectors:Anderson_2_Vertical_Sidy_by_Side" H 9900 3700 60  0001 C CNN
 F 3 "" H 9900 3700 60  0001 C CNN
 	1    10050 4250
@@
 F 0 "Conn11" V 10000 4950 60  0000 C CNN
 F 1 "AndersonPP" V 9900 4950 60  0000 C CNN
-F 2 "MRDT_Connectors:Anderson_2_Horizontal_Side_by_Side_PV" H 9900 4300 60  0001 C CNN
+F 2 "MRDT_Connectors:Anderson_2_Vertical_Sidy_by_Side" H 9900 4300 60  0001 C CNN
 F 3 "" H 9900 4300 60  0001 C CNN
 	1    10050 4850
@@
 F 0 "Conn12" V 10000 5550 60  0000 C CNN
 F 1 "AndersonPP" V 9900 5550 60  0000 C CNN
-F 2 "MRDT_Connectors:Anderson_2_Horizontal_Side_by_Side_PV" H 9900 4900 60  0001 C CNN
+F 2 "MRDT_Connectors:Anderson_2_Vertical_Sidy_by_Side" H 9900 4900 60  0001 C CNN
 F 3 "" H 9900 4900 60  0001 C CNN
 	1    10050 5450
@@
 F 0 "Conn5" V 9450 1200 60  0000 L CNN
 F 1 "AndersonPP" V 9350 1100 60  0000 L CNN
-F 2 "MRDT_Connectors:Anderson_2_Horizontal_Side_by_Side_PV" H 9350 700 60  0001 C CNN
+F 2 "MRDT_Connectors:Anderson_2_Vertical_Sidy_by_Side" H 9350 700 60  0001 C CNN
 F 3 "" H 9350 700 60  0001 C CNN
 	4    9500 1250
@@
 F 0 "Conn6" V 9450 1800 60  0000 L CNN
 F 1 "AndersonPP" V 9350 1700 60  0000 L CNN
-F 2 "MRDT_Connectors:Anderson_2_Horizontal_Side_by_Side_PV" H 9350 1300 60  0001 C CNN
+F 2 "MRDT_Connectors:Anderson_2_Vertical_Sidy_by_Side" H 9350 1300 60  0001 C CNN
 F 3 "" H 9350 1300 60  0001 C CNN
 	4    9500 1850
@@
 F 0 "Conn7" V 9450 2400 60  0000 L CNN
 F 1 "AndersonPP" V 9350 2300 60  0000 L CNN
-F 2 "MRDT_Connectors:Anderson_2_Horizontal_Side_by_Side_PV" H 9350 1900 60  0001 C CNN
+F 2 "MRDT_Connectors:Anderson_2_Vertical_Sidy_by_Side" H 9350 1900 60  0001 C CNN
 F 3 "" H 9350 1900 60  0001 C CNN
 	4    9500 2450
@@
 F 0 "Conn8" V 9450 3000 60  0000 L CNN
 F 1 "AndersonPP" V 9350 2900 60  0000 L CNN
-F 2 "MRDT_Connectors:Anderson_2_Horizontal_Side_by_Side_PV" H 9350 2500 60  0001 C CNN
+F 2 "MRDT_Connectors:Anderson_2_Vertical_Sidy_by_Side" H 9350 2500 60  0001 C CNN
 F 3 "" H 9350 2500 60  0001 C CNN
 	4    9500 3050
@@
 F 0 "Conn8" V 10000 3150 60  0000 C CNN
 F 1 "AndersonPP" V 9900 3150 60  0000 C CNN
-F 2 "MRDT_Connectors:Anderson_2_Horizontal_Side_by_Side_PV" H 9900 2500 60  0001 C CNN
+F 2 "MRDT_Connectors:Anderson_2_Vertical_Sidy_by_Side" H 9900 2500 60  0001 C CNN
 F 3 "" H 9900 2500 60  0001 C CNN
 	1    10050 3050
@@
 F 0 "Conn10" V 9450 4200 60  0000 L CNN
 F 1 "AndersonPP" V 9350 4100 60  0000 L CNN
-F 2 "MRDT_Connectors:Anderson_2_Horizontal_Side_by_Side_PV" H 9350 3700 60  0001 C CNN
+F 2 "MRDT_Connectors:Anderson_2_Vertical_Sidy_by_Side" H 9350 3700 60  0001 C CNN
 F 3 "" H 9350 3700 60  0001 C CNN
 	4    9500 4250
@@
 F 0 "Conn11" V 9450 4800 60  0000 L CNN
 F 1 "AndersonPP" V 9350 4700 60  0000 L CNN
-F 2 "MRDT_Connectors:Anderson_2_Horizontal_Side_by_Side_PV" H 9350 4300 60  0001 C CNN
+F 2 "MRDT_Connectors:Anderson_2_Vertical_Sidy_by_Side" H 9350 4300 60  0001 C CNN
 F 3 "" H 9350 4300 60  0001 C CNN
 	4    9500 4850
@@
 F 0 "Conn12" V 9450 5400 60  0000 L CNN
 F 1 "AndersonPP" V 9350 5300 60  0000 L CNN
-F 2 "MRDT_Connectors:Anderson_2_Horizontal_Side_by_Side_PV" H 9350 4900 60  0001 C CNN
+F 2 "MRDT_Connectors:Anderson_2_Vertical_Sidy_by_Side" H 9350 4900 60  0001 C CNN
 F 3 "" H 9350 4900 60  0001 C CNN
 	4    9500 5450
@@
 F 0 "Conn9" H 10200 3600 60  0000 C CNN
 F 1 "AndersonPP" V 10000 3750 60  0000 C CNN
-F 2 "MRDT_Connectors:Anderson_3_Horizontal_Side_by_Side" H 9900 3100 60  0001 C CNN
+F 2 "MRDT_Connectors:Anderson_3_Vertical_Side_by_Side" H 9900 3100 60  0001 C CNN
 F 3 "" H 9900 3100 60  0001 C CNN
 	2    10050 3650

Commit message: Lots of Changes
Parts:
- removed unit 4 of Conn10
- removed unit 4 of Conn11
- removed unit 4 of Conn12
- removed unit 4 of Conn5
- removed unit 4 of Conn6
- removed unit 4 of Conn7
- removed unit 4 of Conn8
- added Conn10: AndersonPP, MRDT_Connectors:Anderson_2_Vertical_Sidy_by_Side, symbol MRDT_Connectors:AndersonPP
- added unit 2 of Conn2
- added unit 3 of Conn3
- added unit 3 of Conn4
- added unit 2 of Conn5
- added unit 2 of Conn6
- added unit 2 of Conn7
- added unit 3 of Conn8
- added unit 3 of Conn9
- Conn9: footprint MRDT_Connectors:Anderson_3_Vertical_Side_by_Side -> MRDT_Connectors:Anderson_2_Vertical_Sidy_by_Side
- renumbered Conn4 to Conn1, Conn1 to Conn11, Conn5 to Conn2, Conn6 to Conn3, Conn7 to Conn4, Conn8 to Conn5, Conn9 to Conn6, Conn10 to Conn7, Conn11 to Conn8, Conn12 to Conn9
Connections:
- net labels added: "Rev69", Current_Sense_AuxAct, Current_Sense_Gim, Current_Sense_Spare, Driver_AuxAct, Driver_Gim, Driver_Spare
- net labels removed: "Rev4", Anderson_AuxLog, Anderson_BBB, Anderson_Cam1, Anderson_Cam2, Anderson_Drive, Anderson_GimAct, Anderson_GimLog, Anderson_Multi, Anderson_Nav, Anderson_NetSwitch, Anderson_SciAct, Anderson_SciLog, Current_Sense_GimAct, Current_Sense_GimLog, Driver_GimAct, Driver_GimLog
- wire segments 141 -> 127
Other:
- moved on the sheet: Conn11A, Conn11D, Conn9A, Conn9B

Commit message: Fixed schematic and fixed annotations
Parts:
- removed C2: 22uF, Capacitor_THT:CP_Radial_D6.3mm_P2.50mm, symbol Device:CP1
- removed C4: 10uF, Capacitor_SMD:C_0603_1608Metric_Pad1.08x0.95mm_HandSolder, symbol Device:C
- removed C6: 47uF, Capacitor_THT:CP_Radial_D6.3mm_P2.50mm, symbol Device:CP1
- removed D2: LED, Diode_SMD:D_0603_1608Metric_Pad1.05x0.95mm_HandSolder, symbol Device:D
- removed R2: 330, Resistor_SMD:R_0603_1608Metric_Pad0.98x0.95mm_HandSolder, symbol Device:R
- removed U2: OKI-78SR-3.3_1.5-W36-C, Converter_DCDC:Converter_DCDC_muRata_OKI-78SR_Vertical, symbol Converter_DCDC:OKI-78SR-5_1.5-W36-C
- R1: value 510 -> 330
- renumbered C3 to C2, C5 to C3, Conn7 to Conn10, Conn8 to Conn11, Conn9 to Conn12, Conn2 to Conn18, Conn3 to Conn19, Conn11 to Conn2, Conn10 to Conn3, Conn1 to Conn4, Conn2 to Conn5, Conn3 to Conn6, Conn4 to Conn7, Conn5 to Conn8, Conn6 to Conn9
Other:
- moved on the sheet: C1, C2, C3, Conn2A, Conn2D, D1, R1, U1
