File: Hardware/2022_Rev2/12V.sch (KiCad schematic (older format))
At the start: 18 parts, among them Q1 BUK768R3-60E, Q2 BUK768R3-60E, U5 LT1910, U6 LT1910, U7 INA281, U8 INA281

Commit message: Finished footprint signatures and started schematic
Parts:
- R10, R9: footprint (none) -> Resistor_SMD:R_2512_6332Metric_Pad1.40x3.35mm_HandSolder
- R5, R6, R7, R8: footprint (none) -> Resistor_SMD:R_0603_1608Metric_Pad0.98x0.95mm_HandSolder
- U5, U6: footprint (none) -> Package_SO:SOIC-8_3.9x4.9mm_P1.27mm
Changed lines of the file:
@@
 F 0 "R6" V 7600 3000 50  0000 C CNN
 F 1 "5.1k" V 7500 3000 50  0000 C CNN
-F 2 "" V 7430 3000 50  0001 C CNN
+F 2 "Resistor_SMD:R_0603_1608Metric_Pad0.98x0.95mm_HandSolder" V 7430 3000 50  0001 C CNN
 F 3 "~" H 7500 3000 50  0001 C CNN
 	1    7500 3000
@@
 F 0 "U6" H 8575 4087 60  0000 C CNN
 F 1 "LT1910" H 8575 3981 60  0000 C CNN
-F 2 "" H 8200 3400 60  0001 C CNN
+F 2 "Package_SO:SOIC-8_3.9x4.9mm_P1.27mm" H 8200 3400 60  0001 C CNN
 F 3 "" H 8200 3400 60  0001 C CNN
 	1    8200 3400
@@
 F 0 "R8" V 10000 3850 50  0000 C CNN
 F 1 "330" V 10100 3850 50  0000 C CNN
-F 2 "" V 10030 3850 50  0001 C CNN
+F 2 "Resistor_SMD:R_0603_1608Metric_Pad0.98x0.95mm_HandSolder" V 10030 3850 50  0001 C CNN
 F 3 "~" H 10100 3850 50  0001 C CNN
 	1    10100 3850
@@
 F 0 "R10" H 10250 3300 50  0000 L CNN
 F 1 "0.0025" V 10200 3150 50  0000 L CNN
-F 2 "" V 10130 3250 50  0001 C CNN
+F 2 "Resistor_SMD:R_2512_6332Metric_Pad1.40x3.35mm_HandSolder" V 10130 3250 50  0001 C CNN
 F 3 "~" H 10200 3250 50  0001 C CNN
 	1    10200 3250
@@
 F 0 "R5" V 7550 5000 50  0000 C CNN
 F 1 "5.1k" V 7450 5000 50  0000 C CNN
-F 2 "" V 7380 5000 50  0001 C CNN
+F 2 "Resistor_SMD:R_0603_1608Metric_Pad0.98x0.95mm_HandSolder" V 7380 5000 50  0001 C CNN
 F 3 "~" H 7450 5000 50  0001 C CNN
 	1    7450 5000
@@
 F 0 "U5" H 8525 6087 60  0000 C CNN
 F 1 "LT1910" H 8525 5981 60  0000 C CNN
-F 2 "" H 8150 5400 60  0001 C CNN
+F 2 "Package_SO:SOIC-8_3.9x4.9mm_P1.27mm" H 8150 5400 60  0001 C CNN
 F 3 "" H 8150 5400 60  0001 C CNN
 	1    8150 5400
@@
 F 0 "R7" V 9950 5850 50  0000 C CNN
 F 1 "330" V 10050 5850 50  0000 C CNN
-F 2 "" V 9980 5850 50  0001 C CNN
+F 2 "Resistor_SMD:R_0603_1608Metric_Pad0.98x0.95mm_HandSolder" V 9980 5850 50  0001 C CNN
 F 3 "~" H 10050 5850 50  0001 C CNN
 	1    10050 5850
@@
 F 0 "R9" H 10200 5300 50  0000 L CNN
 F 1 "0.0025" V 10150 5150 50  0000 L CNN
-F 2 "" V 10080 5250 50  0001 C CNN
+F 2 "Resistor_SMD:R_2512_6332Metric_Pad1.40x3.35mm_HandSolder" V 10080 5250 50  0001 C CNN
 F 3 "~" H 10150 5250 50  0001 C CNN
 	1    10150 5250

Commit message: Lots of Changes
Parts:
- removed C14: 0.1uF, Capacitor_SMD:C_0603_1608Metric_Pad1.08x0.95mm_HandSolder, symbol Device:C
- removed C16: 10uF, Capacitor_SMD:C_0603_1608Metric_Pad1.08x0.95mm_HandSolder, symbol Device:C
- removed D6: LED, Diode_SMD:D_0603_1608Metric_Pad1.05x0.95mm_HandSolder, symbol Device:D
- removed Q2: BUK768R3-60E, Package_TO_SOT_SMD:LFPAK33, symbol Transistor_FET:BUK7M9R9-60EX
- removed R10: 0.0025, Resistor_SMD:R_2512_6332Metric_Pad1.40x3.35mm_HandSolder, symbol Device:R
- removed R6: 5.1k, Resistor_SMD:R_0603_1608Metric_Pad0.98x0.95mm_HandSolder, symbol Device:R
- removed R8: 330, Resistor_SMD:R_0603_1608Metric_Pad0.98x0.95mm_HandSolder, symbol Device:R
- removed U6: LT1910, Package_SO:SOIC-8_3.9x4.9mm_P1.27mm, symbol 2022_Rev2-rescue:LT1910-MRDT_ICs
- removed U8: INA281, Package_TO_SOT_SMD:SOT-23-5, symbol 2022_Rev2-rescue:INA281-MRDT_ICs
- added F? (x5): 750 mA, symbol Device:Polyfuse_Small
Connections:
- net Anderson_BBB: now also F?.1
- net Anderson_Drive: now also F?.1
- net Anderson_GimAct: now also F?.2
- net Anderson_GimLog: now also F?.1
- net Anderson_Nav: now also F?.1
- new net Anderson_MultiAct: F?.2
- new net Anderson_MultiLog: F?.1
- new net Low Current Out/Anderson_BBB: F?.2
- new net Low Current Out/Anderson_Drive: F?.2
- new net Low Current Out/Anderson_Nav: F?.2

Commit message: Fixed schematic and fixed annotations
Parts:
- gave numbers to parts that had none: 5
- renumbered C13 to C12, C15 to C13, Q1 to Q2, R5 to R7, R7 to R8, U5 to U6
Connections:
- net 12VA: no longer C13.1, Q2.5 (D), U6.6 (SENSE), U6.8 (V+)
- net 5V renamed +5V
- new net +12VA: C13.1, Q2.5 (D), U6.6 (SENSE), U6.8 (V+)
Changed lines of the file:
@@
 $Descr A4 11693 8268
 encoding utf-8
-Sheet 2 4
+Sheet 3 4
 Title ""
 Date ""
@@
 Comment4 ""
 $EndDescr
-Text HLabel 1350 1000 0    50   Input ~ 0
-5V
 Text HLabel 1350 1750 0    50   Input ~ 0
 Driver_Nav
-Wire Wire Line
-	1350 1000 1450 1000
 Wire Wire Line
 	1450 1750 1350 1750
@@
 AR Path="/62118E70/621219B0/624A08A6" Ref="R?"  Part="1"
 AR Path="/62118E70/622EFCD1/624A08A6" Ref="R?"  Part="1"
-AR Path="/62118E70/624A08A6" Ref="R5"  Part="1"
-F 0 "R5" V 7550 5000 50  0000 C CNN
+AR Path="/62118E70/624A08A6" Ref="R7"  Part="1"
+F 0 "R7" V 7550 5000 50  0000 C CNN
 F 1 "5.1k" V 7450 5000 50  0000 C CNN
 F 2 "Resistor_SMD:R_0603_1608Metric_Pad0.98x0.95mm_HandSolder" V 7380 5000 50  0001 C CNN
@@
 AR Path="/62118E70/621219B0/624A08AC" Ref="U?"  Part="1"
 AR Path="/62118E70/622EFCD1/624A08AC" Ref="U?"  Part="1"
-AR Path="/62118E70/624A08AC" Ref="U5"  Part="1"
-F 0 "U5" H 8525 6087 60  0000 C CNN
+AR Path="/62118E70/624A08AC" Ref="U6"  Part="1"
+F 0 "U6" H 8525 6087 60  0000 C CNN
 F 1 "LT1910" H 8525 5981 60  0000 C CNN
 F 2 "Package_SO:SOIC-8_3.9x4.9mm_P1.27mm" H 8150 5400 60  0001 C CNN
@@
 AR Path="/62118E70/621219B0/624A08B2" Ref="C?"  Part="1"
 AR Path="/62118E70/622EFCD1/624A08B2" Ref="C?"  Part="1"
-AR Path="/62118E70/624A08B2" Ref="C13"  Part="1"
-F 0 "C13" H 8065 5746 50  0000 L CNN
+AR Path="/62118E70/624A08B2" Ref="C12"  Part="1"
+F 0 "C12" H 8065 5746 50  0000 L CNN
 F 1 "0.1uF" H 8065 5655 50  0000 L CNN
 F 2 "Capacitor_SMD:C_0603_1608Metric_Pad1.08x0.95mm_HandSolder" H 7988 5550 50  0001 C CNN
@@
 AR Path="/62118E70/621219B0/624A08B8" Ref="#PWR?"  Part="1"
 AR Path="/62118E70/622EFCD1/624A08B8" Ref="#PWR?"  Part="1"
-AR Path="/62118E70/624A08B8" Ref="#PWR0121"  Part="1"
-F 0 "#PWR0121" H 8550 5600 50  0001 C CNN
+AR Path="/62118E70/624A08B8" Ref="#PWR033"  Part="1"
+F 0 "#PWR033" H 8550 5600 50  0001 C CNN
 F 1 "GND" H 8555 5677 50  0000 C CNN
 F 2 "" H 8550 5850 50  0001 C CNN
@@
 AR Path="/62118E70/621219B0/624A08BE" Ref="C?"  Part="1"
 AR Path="/62118E70/622EFCD1/624A08BE" Ref="C?"  Part="1"
-AR Path="/62118E70/624A08BE" Ref="C15"  Part="1"
-F 0 "C15" H 9315 5646 50  0000 L CNN
+AR Path="/62118E70/624A08BE" Ref="C13"  Part="1"
+F 0 "C13" H 9315 5646 50  0000 L CNN
 F 1 "10uF" H 9315 5555 50  0000 L CNN
 F 2 "Capacitor_SMD:C_0603_1608Metric_Pad1.08x0.95mm_HandSolder" H 9238 5450 50  0001 C CNN
@@
 AR Path="/62118E70/621219B0/624A08C4" Ref="Q?"  Part="1"
 AR Path="/62118E70/622EFCD1/624A08C4" Ref="Q?"  Part="1"
-AR Path="/62118E70/624A08C4" Ref="Q1"  Part="1"
-F 0 "Q1" H 9800 5050 50  0000 L CNN
+AR Path="/62118E70/624A08C4" Ref="Q2"  Part="1"
+F 0 "Q2" H 9800 5050 50  0000 L CNN
 F 1 "BUK768R3-60E" H 9350 4950 50  0000 L CNN
 F 2 "Package_TO_SOT_SMD:LFPAK33" H 9850 5125 50  0001 L CIN
@@
 AR Path="/62118E70/621219B0/624A08CA" Ref="R?"  Part="1"
 AR Path="/62118E70/622EFCD1/624A08CA" Ref="R?"  Part="1"
-AR Path="/62118E70/624A08CA" Ref="R7"  Part="1"
-F 0 "R7" V 9950 5850 50  0000 C CNN
+AR Path="/62118E70/624A08CA" Ref="R8"  Part="1"
+F 0 "R8" V 9950 5850 50  0000 C CNN
 F 1 "330" V 10050 5850 50  0000 C CNN
 F 2 "Resistor_SMD:R_0603_1608Metric_Pad0.98x0.95mm_HandSolder" V 9980 5850 50  0001 C CNN
@@
 AR Path="/62118E70/621219B0/624A08F2" Ref="#PWR?"  Part="1"
 AR Path="/62118E70/622EFCD1/624A08F2" Ref="#PWR?"  Part="1"
-AR Path="/62118E70/624A08F2" Ref="#PWR0122"  Part="1"
-F 0 "#PWR0122" H 10700 5750 50  0001 C CNN
+AR Path="/62118E70/624A08F2" Ref="#PWR037"  Part="1"
+F 0 "#PWR037" H 10700 5750 50  0001 C CNN
 F 1 "GND" H 10705 5827 50  0000 C CNN
 F 2 "" H 10700 6000 50  0001 C CNN
@@
 AR Path="/62118E70/621219B0/624A090A" Ref="#PWR?"  Part="1"
 AR Path="/62118E70/622EFCD1/624A090A" Ref="#PWR?"  Part="1"
-AR Path="/62118E70/624A090A" Ref="#PWR0123"  Part="1"
-F 0 "#PWR0123" H 10600 5250 50  0001 C CNN
+AR Path="/62118E70/624A090A" Ref="#PWR036"  Part="1"
+F 0 "#PWR036" H 10600 5250 50  0001 C CNN
 F 1 "GND" H 10605 5327 50  0000 C CNN
 F 2 "" H 10600 5500 50  0001 C CNN
@@
 Text HLabel 7600 5150 3    50   Input ~ 0
 Driver_AuxLog
-Text HLabel 7200 4850 1    50   Input ~ 0
-5V
-Text HLabel 10600 4750 0    50   Input ~ 0
-5V
 Wire Wire Line
 	9200 5000 9200 4550
 Wire Wire Line
 	9200 4550 9000 4550
-Text HLabel 9000 4550 0    50   Input ~ 0
-12VA
 Text Notes 7250 4550 0    50   ~ 0
 3 amps for SciLog, SciAct, and Aux
@@
 	5400 2400 5750 2400
 $Comp
-L Device:Polyfuse_Small F?
+L Device:Polyfuse_Small F4
 U 1 1 62482698
 P 5600 2600
-F 0 "F?" V 5395 2600 50  0000 C CNN
+F 0 "F4" V 5395 2600 50  0000 C CNN
 F 1 "750 mA" V 5486 2600 50  0000 C CNN
 F 2 "" H 5650 2400 50  0001 L CNN
@@
 $EndComp
 $Comp
-L Device:Polyfuse_Small F?
+L Device:Polyfuse_Small F5
 U 1 1 62482E09
 P 5600 2900
-F 0 "F?" V 5395 2900 50  0000 C CNN
+F 0 "F5" V 5395 2900 50  0000 C CNN
 F 1 "750 mA" V 5486 2900 50  0000 C CNN
 F 2 "" H 5650 2700 50  0001 L CNN
@@
 	3750 2700 5400 2700
 $Comp
-L Device:Polyfuse_Small F?
+L Device:Polyfuse_Small F2
 U 1 1 62494A24
 P 3950 2500
-F 0 "F?" V 3900 2500 50  0000 C CNN
+F 0 "F2" V 3900 2500 50  0000 C CNN
 F 1 "750 mA" V 4000 2500 50  0000 C CNN
 F 2 "" H 4000 2300 50  0001 L CNN
@@
 	4050 2500 4150 2500
 $Comp
-L Device:Polyfuse_Small F?
+L Device:Polyfuse_Small F3
 U 1 1 62497059
 P 3950 2800
-F 0 "F?" V 3900 2800 50  0000 C CNN
+F 0 "F3" V 3900 2800 50  0000 C CNN
 F 1 "750 mA" V 4000 2800 50  0000 C CNN
 F 2 "" H 4000 2600 50  0001 L CNN
@@
 	4050 2800 4150 2800
 $Comp
-L Device:Polyfuse_Small F?
+L Device:Polyfuse_Small F1
 U 1 1 6249917B
 P 3950 2200
-F 0 "F?" V 3900 2200 50  0000 C CNN
+F 0 "F1" V 3900 2200 50  0000 C CNN
 F 1 "750 mA" V 4000 2200 50  0000 C CNN
 F 2 "" H 4000 2000 50  0001 L CNN
@@
 F0 "Low Current Out" 50
 F1 "Low Current Out.sch" 50
-F2 "5V" I L 1450 1000 50
-F3 "Current_Sense_Drive" O R 3750 1450 50
-F4 "Anderson_Drive" O R 3750 2500 50
-F5 "Driver_Drive" I L 1450 1450 50
-F6 "Current_Sense_Nav" O R 3750 1750 50
-F7 "Anderson_Nav" O R 3750 2800 50
-F8 "Driver_Nav" I L 1450 1750 50
-F9 "Current_Sense_BBB" O R 3750 1150 50
-F10 "Anderson_BBB" O R 3750 2200 50
-F11 "Current_Sense_Multi" O R 3750 1650 50
-F12 "Anderson_Multi" O R 3750 2700 50
-F13 "Current_Sense_Cam1" O R 3750 1250 50
-F14 "Anderson_Cam1" O R 3750 2300 50
-F15 "Driver_Cam1" I L 1450 1250 50
-F16 "Current_Sense_NetSwitch" O R 3750 1850 50
-F17 "Anderson_NetSwitch" O R 3750 2900 50
-F18 "Current_Sense_Cam2" O R 3750 1350 50
-F19 "Anderson_Cam2" O R 3750 2400 50
-F20 "Driver_Cam2" I L 1450 1350 50
-F21 "Driver_BBB" I L 1450 1150 50
-F22 "Driver_Multi" I L 1450 1650 50
-F23 "Current_Sense_Gim" O R 3750 1550 50
-F24 "Anderson_Gim" O R 3750 2600 50
-F25 "Driver_Gim" I L 1450 1550 50
-F26 "Driver_NetSwitch" I L 1450 1850 50
-F27 "12VA" I L 1450 1950 50
-F28 "Current_Sense_Spare" O R 3750 1950 50
-F29 "Anderson_Spare" O R 3750 3000 50
-F30 "Driver_Spare" I L 1450 2050 50
+F2 "Current_Sense_Drive" O R 3750 1450 50
+F3 "Anderson_Drive" O R 3750 2500 50
+F4 "Driver_Drive" I L 1450 1450 50
+F5 "Current_Sense_Nav" O R 3750 1750 50
+F6 "Anderson_Nav" O R 3750 2800 50
+F7 "Driver_Nav" I L 1450 1750 50
+F8 "Current_Sense_BBB" O R 3750 1150 50
+F9 "Anderson_BBB" O R 3750 2200 50
+F10 "Current_Sense_Multi" O R 3750 1650 50
+F11 "Anderson_Multi" O R 3750 2700 50
+F12 "Current_Sense_Cam1" O R 3750 1250 50
+F13 "Anderson_Cam1" O R 3750 2300 50
+F14 "Driver_Cam1" I L 1450 1250 50
+F15 "Current_Sense_NetSwitch" O R 3750 1850 50
+F16 "Anderson_NetSwitch" O R 3750 2900 50
+F17 "Current_Sense_Cam2" O R 3750 1350 50
+F18 "Anderson_Cam2" O R 3750 2400 50
+F19 "Driver_Cam2" I L 1450 1350 50
+F20 "Driver_BBB" I L 1450 1150 50
+F21 "Driver_Multi" I L 1450 1650 50
+F22 "Current_Sense_Gim" O R 3750 1550 50
+F23 "Anderson_Gim" O R 3750 2600 50
+F24 "Driver_Gim" I L 1450 1550 50
+F25 "Driver_NetSwitch" I L 1450 1850 50
+F26 "12VA" I L 1450 1950 50
+F27 "Current_Sense_Spare" O R 3750 1950 50
+F28 "Anderson_Spare" O R 3750 3000 50
+F29 "Driver_Spare" I L 1450 2050 50
 $EndSheet
 Text HLabel 3850 1950 2    50   Output ~ 0
@@
 Wire Wire Line
 	1350 2050 1450 2050
+$Comp
+L power:+5V #PWR032
+U 1 1 627B9AAD
+P 7200 4850
+F 0 "#PWR032" H 7200 4700 50  0001 C CNN
+F 1 "+5V" H 7215 5023 50  0000 C CNN
+F 2 "" H 7200 4850 50  0001 C CNN
+F 3 "" H 7200 4850 50  0001 C CNN
+	1    7200 4850
+	1    0    0    -1
+$EndComp
+$Comp
+L power:+5V #PWR035
+U 1 1 627B9F25
+P 10600 4750
+F 0 "#PWR035" H 10600 4600 50  0001 C CNN
+F 1 "+5V" H 10615 4923 50  0000 C CNN
+F 2 "" H 10600 4750 50  0001 C CNN
+F 3 "" H 10600 4750 50  0001 C CNN
+	1    10600 4750
+	1    0    0    -1
+$EndComp
+$Comp
+L power:+12VA #PWR034
+U 1 1 627C8478
+P 9000 4550
+F 0 "#PWR034" H 9000 4400 50  0001 C CNN
+F 1 "+12VA" H 9015 4723 50  0000 C CNN
+F 2 "" H 9000 4550 50  0001 C CNN
+F 3 "" H 9000 4550 50  0001 C CNN
+	1    9000 4550
+	1    0    0    -1
+$EndComp
 $EndSCHEMATC

Commit message: Assigned footprints and finished changes on schem
Parts:
- F1, F2, F3, F4, F5: footprint (none) -> Fuse:Fuse_2920_7451Metric
Changed lines of the file:
@@
 F 0 "F4" V 5395 2600 50  0000 C CNN
 F 1 "750 mA" V 5486 2600 50  0000 C CNN
-F 2 "" H 5650 2400 50  0001 L CNN
+F 2 "Fuse:Fuse_2920_7451Metric" H 5650 2400 50  0001 L CNN
 F 3 "~" H 5600 2600 50  0001 C CNN
 	1    5600 2600
@@
 F 0 "F5" V 5395 2900 50  0000 C CNN
 F 1 "750 mA" V 5486 2900 50  0000 C CNN
-F 2 "" H 5650 2700 50  0001 L CNN
+F 2 "Fuse:Fuse_2920_7451Metric" H 5650 2700 50  0001 L CNN
 F 3 "~" H 5600 2900 50  0001 C CNN
 	1    5600 2900
@@
 F 0 "F2" V 3900 2500 50  0000 C CNN
 F 1 "750 mA" V 4000 2500 50  0000 C CNN
-F 2 "" H 4000 2300 50  0001 L CNN
+F 2 "Fuse:Fuse_2920_7451Metric" H 4000 2300 50  0001 L CNN
 F 3 "~" H 3950 2500 50  0001 C CNN
 	1    3950 2500
@@
 F 0 "F3" V 3900 2800 50  0000 C CNN
 F 1 "750 mA" V 4000 2800 50  0000 C CNN
-F 2 "" H 4000 2600 50  0001 L CNN
+F 2 "Fuse:Fuse_2920_7451Metric" H 4000 2600 50  0001 L CNN
 F 3 "~" H 3950 2800 50  0001 C CNN
 	1    3950 2800
@@
 F 0 "F1" V 3900 2200 50  0000 C CNN
 F 1 "750 mA" V 4000 2200 50  0000 C CNN
-F 2 "" H 4000 2000 50  0001 L CNN
+F 2 "Fuse:Fuse_2920_7451Metric" H 4000 2000 50  0001 L CNN
 F 3 "~" H 3950 2200 50  0001 C CNN
 	1    3950 2200

Commit message: Fixed many issues
Parts:
- removed C12: 0.1uF, Capacitor_SMD:C_0603_1608Metric_Pad1.08x0.95mm_HandSolder, symbol Device:C
- removed C13: 10uF, Capacitor_SMD:C_0603_1608Metric_Pad1.08x0.95mm_HandSolder, symbol Device:C
- removed D5: LED, Diode_SMD:D_0603_1608Metric_Pad1.05x0.95mm_HandSolder, symbol Device:D
- removed F1, F2, F3, F4, F5: 750 mA, Fuse:Fuse_2920_7451Metric, symbol Device:Polyfuse_Small
- removed Q2: BUK768R3-60E, Package_TO_SOT_SMD:LFPAK33, symbol Transistor_FET:BUK7M9R9-60EX
- removed R7: 5.1k, Resistor_SMD:R_0603_1608Metric_Pad0.98x0.95mm_HandSolder, symbol Device:R
- removed R8: 330, Resistor_SMD:R_0603_1608Metric_Pad0.98x0.95mm_HandSolder, symbol Device:R
- removed R9: 0.0025, Resistor_SMD:R_2512_6332Metric_Pad1.40x3.35mm_HandSolder, symbol Device:R
- removed U6: LT1910, Package_SO:SOIC-8_3.9x4.9mm_P1.27mm, symbol 2022_Rev2-rescue:LT1910-MRDT_ICs
- removed U7: INA281, Package_TO_SOT_SMD:SOT-23-5, symbol 2022_Rev2-rescue:INA281-MRDT_ICs
Other:
- note removed: "3 amps for SciLog, SciAct, and Aux"

Commit message: ahhhhhh ladybug is angy
Changed lines of the file:
@@
 Wire Wire Line
 	3750 1650 3850 1650
-Text HLabel 3850 1850 2    50   Output ~ 0
-Current_Sense_NetSwitch
-Wire Wire Line
-	3750 1850 3850 1850
 Text HLabel 4150 2200 2    50   Output ~ 0
 Anderson_BBB
@@
 Wire Wire Line
 	1350 1650 1450 1650
-Text HLabel 1350 1850 0    50   Input ~ 0
-Driver_NetSwitch
-Wire Wire Line
-	1350 1850 1450 1850
 Text HLabel 5750 2600 2    50   Output ~ 0
 Anderson_GimLog
@@
 F13 "Anderson_Cam1" O R 3750 2300 50
 F14 "Driver_Cam1" I L 1450 1250 50
-F15 "Current_Sense_NetSwitch" O R 3750 1850 50
-F16 "Anderson_NetSwitch" O R 3750 2900 50
-F17 "Current_Sense_Cam2" O R 3750 1350 50
-F18 "Anderson_Cam2" O R 3750 2400 50
-F19 "Driver_Cam2" I L 1450 1350 50
-F20 "Driver_BBB" I L 1450 1150 50
-F21 "Driver_Multi" I L 1450 1650 50
-F22 "Current_Sense_Gim" O R 3750 1550 50
-F23 "Anderson_Gim" O R 3750 2600 50
-F24 "Driver_Gim" I L 1450 1550 50
-F25 "Driver_NetSwitch" I L 1450 1850 50
-F26 "Current_Sense_Spare" O R 3750 1950 50
-F27 "Anderson_Spare" O R 3750 3000 50
-F28 "Driver_Spare" I L 1450 2050 50
+F15 "Anderson_NetSwitch" O R 3750 2900 50
+F16 "Current_Sense_Cam2" O R 3750 1350 50
+F17 "Anderson_Cam2" O R 3750 2400 50
+F18 "Driver_Cam2" I L 1450 1350 50
+F19 "Driver_BBB" I L 1450 1150 50
+F20 "Driver_Multi" I L 1450 1650 50
+F21 "Current_Sense_Gim" O R 3750 1550 50
+F22 "Anderson_Gim" O R 3750 2600 50
+F23 "Driver_Gim" I L 1450 1550 50
+F24 "Current_Sense_Spare" O R 3750 1950 50
+F25 "Anderson_Spare" O R 3750 3000 50
+F26 "Driver_Spare" I L 1450 2050 50
 $EndSheet
 Text HLabel 3850 1950 2    50   Output ~ 0
@@
 	3850 1950 3750 1950
 Text HLabel 3850 3000 2    50   Output ~ 0
-Anderson_Spare_Logic
+Anderson_Spare
 Wire Wire Line
 	3850 3000 3750 3000
