File: Hardware/2022_Rev2/Low Current Out.sch (KiCad schematic (older format))
At the start: 77 parts, among them Q10 BUK768R3-60E, Q11 BUK768R3-60E, Q3 BUK768R3-60E, Q4 BUK768R3-60E, Q6 BUK768R3-60E, Q7 BUK768R3-60E, Q8 BUK768R3-60E, Q9 BUK768R3-60E, U11 LT1910, U12 INA281, U13 INA281, U15 INA281, U16 INA281, U17 LT1910, U18 LT1910, U19 INA281, U20 LT1910, U21 LT1910, U22 LT1910, U23 INA281, U24 INA281, U25 INA281, U8 LT1910, U9 LT1910

Commit message: ahhhhhh ladybug is angy
Parts:
- Q10, Q3, Q8, Q9: value BUK768R3-60E -> FDC855N; footprint Package_TO_SOT_SMD:LFPAK33 -> Package_TO_SOT_SMD:SuperSOT-6
- Q11, Q4, Q6, Q7: value BUK768R3-60E -> IRLML2803TRPBF; footprint Package_TO_SOT_SMD:LFPAK33 -> Package_TO_SOT_SMD:SOT-23
- R16, R18, R21, R23, R26, R34, R35, R36: value 0.0025 -> 0.003; footprint Resistor_SMD:R_2512_6332Metric_Pad1.40x3.35mm_HandSolder -> Resistor_SMD:R_2010_5025Metric_Pad1.52x2.65mm_HandSolder
Changed lines of the file:
@@
 P 3100 4850
 F 0 "Q6" H 3250 4700 50  0000 L CNN
-F 1 "BUK768R3-60E" H 2800 4600 50  0000 L CNN
-F 2 "Package_TO_SOT_SMD:LFPAK33" H 3300 4775 50  0001 L CIN
-F 3 "https://assets.nexperia.com/documents/data-sheet/BUK7M9R9-60E.pdf" V 3100 4850 50  0001 L CNN
+F 1 "IRLML2803TRPBF" H 2800 4600 50  0000 L CNN
+F 2 "Package_TO_SOT_SMD:SOT-23" H 3300 4775 50  0001 L CIN
+F 3 "https://www.infineon.com/dgdl/irlml2803pbf.pdf?fileId=5546d462533600a4015356682aff260f" V 3100 4850 50  0001 L CNN
 	1    3100 4850
 	1    0    0    -1
@@
 P 3600 4900
 F 0 "R21" H 3650 4950 50  0000 L CNN
-F 1 "0.0025" V 3600 4800 50  0000 L CNN
-F 2 "Resistor_SMD:R_2512_6332Metric_Pad1.40x3.35mm_HandSolder" V 3530 4900 50  0001 C CNN
+F 1 "0.003" V 3600 4800 50  0000 L CNN
+F 2 "Resistor_SMD:R_2010_5025Metric_Pad1.52x2.65mm_HandSolder" V 3530 4900 50  0001 C CNN
 F 3 "~" H 3600 4900 50  0001 C CNN
 	1    3600 4900
@@
 P 2950 3050
 F 0 "Q3" H 3100 2900 50  0000 L CNN
-F 1 "BUK768R3-60E" H 2650 2800 50  0000 L CNN
-F 2 "Package_TO_SOT_SMD:LFPAK33" H 3150 2975 50  0001 L CIN
-F 3 "https://assets.nexperia.com/documents/data-sheet/BUK7M9R9-60E.pdf" V 2950 3050 50  0001 L CNN
+F 1 "FDC855N" H 2650 2800 50  0000 L CNN
+F 2 "Package_TO_SOT_SMD:SuperSOT-6" H 3150 2975 50  0001 L CIN
+F 3 "https://www.onsemi.com/pdf/datasheet/fdc855n-d.pdf" V 2950 3050 50  0001 L CNN
 	1    2950 3050
 	1    0    0    -1
@@
 P 3450 3100
 F 0 "R16" H 3500 3150 50  0000 L CNN
-F 1 "0.0025" V 3450 3000 50  0000 L CNN
-F 2 "Resistor_SMD:R_2512_6332Metric_Pad1.40x3.35mm_HandSolder" V 3380 3100 50  0001 C CNN
+F 1 "0.003" V 3450 3000 50  0000 L CNN
+F 2 "Resistor_SMD:R_2010_5025Metric_Pad1.52x2.65mm_HandSolder" V 3380 3100 50  0001 C CNN
 F 3 "~" H 3450 3100 50  0001 C CNN
 	1    3450 3100
@@
 P 3000 1300
 F 0 "Q4" H 3150 1150 50  0000 L CNN
-F 1 "BUK768R3-60E" H 2700 1050 50  0000 L CNN
-F 2 "Package_TO_SOT_SMD:LFPAK33" H 3200 1225 50  0001 L CIN
-F 3 "https://assets.nexperia.com/documents/data-sheet/BUK7M9R9-60E.pdf" V 3000 1300 50  0001 L CNN
+F 1 "IRLML2803TRPBF" H 2700 1050 50  0000 L CNN
+F 2 "Package_TO_SOT_SMD:SOT-23" H 3200 1225 50  0001 L CIN
+F 3 "https://www.infineon.com/dgdl/irlml2803pbf.pdf?fileId=5546d462533600a4015356682aff260f" V 3000 1300 50  0001 L CNN
 	1    3000 1300
 	1    0    0    -1
@@
 P 3500 1350
 F 0 "R18" H 3550 1400 50  0000 L CNN
-F 1 "0.0025" V 3500 1250 50  0000 L CNN
-F 2 "Resistor_SMD:R_2512_6332Metric_Pad1.40x3.35mm_HandSolder" V 3430 1350 50  0001 C CNN
+F 1 "0.003" V 3500 1250 50  0000 L CNN
+F 2 "Resistor_SMD:R_2010_5025Metric_Pad1.52x2.65mm_HandSolder" V 3430 1350 50  0001 C CNN
 F 3 "~" H 3500 1350 50  0001 C CNN
 	1    3500 1350
@@
 P 9750 1400
 F 0 "Q11" H 9900 1250 50  0000 L CNN
-F 1 "BUK768R3-60E" H 9450 1150 50  0000 L CNN
-F 2 "Package_TO_SOT_SMD:LFPAK33" H 9950 1325 50  0001 L CIN
-F 3 "https://assets.nexperia.com/documents/data-sheet/BUK7M9R9-60E.pdf" V 9750 1400 50  0001 L CNN
+F 1 "IRLML2803TRPBF" H 9450 1150 50  0000 L CNN
+F 2 "Package_TO_SOT_SMD:SOT-23" H 9950 1325 50  0001 L CIN
+F 3 "https://www.infineon.com/dgdl/irlml2803pbf.pdf?fileId=5546d462533600a4015356682aff260f" V 9750 1400 50  0001 L CNN
 	1    9750 1400
 	1    0    0    -1
@@
 P 10250 1450
 F 0 "R36" H 10300 1500 50  0000 L CNN
-F 1 "0.0025" V 10250 1350 50  0000 L CNN
-F 2 "Resistor_SMD:R_2512_6332Metric_Pad1.40x3.35mm_HandSolder" V 10180 1450 50  0001 C CNN
+F 1 "0.003" V 10250 1350 50  0000 L CNN
+F 2 "Resistor_SMD:R_2010_5025Metric_Pad1.52x2.65mm_HandSolder" V 10180 1450 50  0001 C CNN
 F 3 "~" H 10250 1450 50  0001 C CNN
 	1    10250 1450
@@
 P 9700 3300
 F 0 "Q9" H 9850 3150 50  0000 L CNN
-F 1 "BUK768R3-60E" H 9400 3050 50  0000 L CNN
-F 2 "Package_TO_SOT_SMD:LFPAK33" H 9900 3225 50  0001 L CIN
-F 3 "https://assets.nexperia.com/documents/data-sheet/BUK7M9R9-60E.pdf" V 9700 3300 50  0001 L CNN
+F 1 "FDC855N" H 9400 3050 50  0000 L CNN
+F 2 "Package_TO_SOT_SMD:SuperSOT-6" H 9900 3225 50  0001 L CIN
+F 3 "https://www.onsemi.com/pdf/datasheet/fdc855n-d.pdf" V 9700 3300 50  0001 L CNN
 	1    9700 3300
 	1    0    0    -1
@@
 P 10200 3350
 F 0 "R34" H 10250 3400 50  0000 L CNN
-F 1 "0.0025" V 10200 3250 50  0000 L CNN
-F 2 "Resistor_SMD:R_2512_6332Metric_Pad1.40x3.35mm_HandSolder" V 10130 3350 50  0001 C CNN
+F 1 "0.003" V 10200 3250 50  0000 L CNN
+F 2 "Resistor_SMD:R_2010_5025Metric_Pad1.52x2.65mm_HandSolder" V 10130 3350 50  0001 C CNN
 F 3 "~" H 10200 3350 50  0001 C CNN
 	1    10200 3350
@@
 P 9700 5100
 F 0 "Q10" H 9850 4950 50  0000 L CNN
-F 1 "BUK768R3-60E" H 9400 4850 50  0000 L CNN
-F 2 "Package_TO_SOT_SMD:LFPAK33" H 9900 5025 50  0001 L CIN
-F 3 "https://assets.nexperia.com/documents/data-sheet/BUK7M9R9-60E.pdf" V 9700 5100 50  0001 L CNN
+F 1 "FDC855N" H 9400 4850 50  0000 L CNN
+F 2 "Package_TO_SOT_SMD:SuperSOT-6" H 9900 5025 50  0001 L CIN
+F 3 "https://www.onsemi.com/pdf/datasheet/fdc855n-d.pdf" V 9700 5100 50  0001 L CNN
 	1    9700 5100
 	1    0    0    -1
@@
 P 10200 5150
 F 0 "R35" H 10250 5200 50  0000 L CNN
-F 1 "0.0025" V 10200 5050 50  0000 L CNN
-F 2 "Resistor_SMD:R_2512_6332Metric_Pad1.40x3.35mm_HandSolder" V 10130 5150 50  0001 C CNN
+F 1 "0.003" V 10200 5050 50  0000 L CNN
+F 2 "Resistor_SMD:R_2010_5025Metric_Pad1.52x2.65mm_HandSolder" V 10130 5150 50  0001 C CNN
 F 3 "~" H 10200 5150 50  0001 C CNN
 	1    10200 5150
@@
 P 6400 6300
 F 0 "Q8" H 6550 6150 50  0000 L CNN
-F 1 "BUK768R3-60E" H 6100 6050 50  0000 L CNN
-F 2 "Package_TO_SOT_SMD:LFPAK33" H 6600 6225 50  0001 L CIN
-F 3 "https://assets.nexperia.com/documents/data-sheet/BUK7M9R9-60E.pdf" V 6400 6300 50  0001 L CNN
+F 1 "FDC855N" H 6100 6050 50  0000 L CNN
+F 2 "Package_TO_SOT_SMD:SuperSOT-6" H 6600 6225 50  0001 L CIN
+F 3 "https://www.onsemi.com/pdf/datasheet/fdc855n-d.pdf" V 6400 6300 50  0001 L CNN
 	1    6400 6300
 	0    1    1    0
@@
 P 6350 6800
 F 0 "R26" H 6400 6850 50  0000 L CNN
-F 1 "0.0025" V 6350 6700 50  0000 L CNN
-F 2 "Resistor_SMD:R_2512_6332Metric_Pad1.40x3.35mm_HandSolder" V 6280 6800 50  0001 C CNN
+F 1 "0.003" V 6350 6700 50  0000 L CNN
+F 2 "Resistor_SMD:R_2010_5025Metric_Pad1.52x2.65mm_HandSolder" V 6280 6800 50  0001 C CNN
 F 3 "~" H 6350 6800 50  0001 C CNN
 	1    6350 6800
@@
 P 5500 2050
 F 0 "Q7" H 5650 1900 50  0000 L CNN
-F 1 "BUK768R3-60E" H 5200 1800 50  0000 L CNN
-F 2 "Package_TO_SOT_SMD:LFPAK33" H 5700 1975 50  0001 L CIN
-F 3 "https://assets.nexperia.com/documents/data-sheet/BUK7M9R9-60E.pdf" V 5500 2050 50  0001 L CNN
+F 1 "IRLML2803TRPBF" H 5200 1800 50  0000 L CNN
+F 2 "Package_TO_SOT_SMD:SOT-23" H 5700 1975 50  0001 L CIN
+F 3 "https://www.infineon.com/dgdl/irlml2803pbf.pdf?fileId=5546d462533600a4015356682aff260f" V 5500 2050 50  0001 L CNN
 	1    5500 2050
 	0    -1   -1   0
@@
 P 5550 1550
 F 0 "R23" H 5600 1600 50  0000 L CNN
-F 1 "0.0025" V 5550 1450 50  0000 L CNN
-F 2 "Resistor_SMD:R_2512_6332Metric_Pad1.40x3.35mm_HandSolder" V 5480 1550 50  0001 C CNN
+F 1 "0.003" V 5550 1450 50  0000 L CNN
+F 2 "Resistor_SMD:R_2010_5025Metric_Pad1.52x2.65mm_HandSolder" V 5480 1550 50  0001 C CNN
 F 3 "~" H 5550 1550 50  0001 C CNN
 	1    5550 1550

Commit message: Gerbs are done
please review before you order this max
Parts:
- removed Q10, Q3, Q8, Q9: FDC855N, Package_TO_SOT_SMD:SuperSOT-6, symbol Transistor_FET:BUK7M9R9-60EX
- removed Q11, Q4, Q6, Q7: IRLML2803TRPBF, Package_TO_SOT_SMD:SOT-23, symbol Transistor_FET:BUK7M9R9-60EX
- added F1: 5A, MRDT_Passives:ATC_Fuse_Block, symbol Device:Fuse
- added Q1, Q3, Q8: IRLML2803TRPBF, Package_TO_SOT_SMD:SOT-23, symbol Transistor_FET:IRLML0030
- added Q2, Q4, Q5, Q6, Q7: FDC855N, Package_TO_SOT_SMD:SuperSOT-6, symbol 12V_6A_Mosfet:FDC855N
- C14, C15, C17, C18, C19, C21, C22, C23, C24, C25, C26, C27, C28, C29, C30, C31: footprint Capacitor_SMD:C_0603_1608Metric_Pad1.08x0.95mm_HandSolder -> Capacitor_SMD:C_0603_1608Metric_Pad1.05x0.95mm_HandSolder
- R10, R11, R13, R14, R15, R17, R19, R22, R24, R25, R27, R28, R29, R30, R31, R32, R33: footprint Resistor_SMD:R_0603_1608Metric_Pad0.98x0.95mm_HandSolder -> Resistor_SMD:R_0603_1608Metric_Pad1.05x0.95mm_HandSolder
Connections:
- net +12VA: now also F1.1, Q1.3 (D), Q3.3 (D), Q8.3 (D); no longer C22.1, U17.6 (SENSE), U17.8 (V+)
- net at U11.5 (GATE): now also Q3.1 (G)
- net at R19.2, R21.1, U15.3 (+): now also Q3.2 (S)
- net at U8.5 (GATE): now also Q2.3 (Gate)
- net at C18.1, F6.2, U8.6 (SENSE)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: now also Q2.1 (Drain), Q2.2 (Drain), Q2.5 (Drain), Q2.6 (Drain)
- net at R14.2, R16.1, U12.3 (+): now also Q2.4 (Source)
- net at U9.5 (GATE): now also Q1.1 (G)
- net at R15.2, R18.1, U13.3 (+): now also Q1.2 (S)
- net at U22.5 (GATE): now also Q8.1 (G)
- net at R33.2, R36.1, U25.3 (+): now also Q8.2 (S)
- net at U20.5 (GATE): now also Q6.3 (Gate)
- net at C29.1, F9.2, U20.6 (SENSE)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: now also Q6.1 (Drain), Q6.2 (Drain), Q6.5 (Drain), Q6.6 (Drain)
- net at R31.2, R34.1, U23.3 (+): now also Q6.4 (Source)
- net at U21.5 (GATE): now also Q7.3 (Gate)
- net at C25.1, C30.1, F8.2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: now also Q5.1 (Drain), Q5.2 (Drain), Q5.5 (Drain), Q5.6 (Drain), Q7.1 (Drain), Q7.2 (Drain), Q7.5 (Drain), Q7.6 (Drain)
- net at R32.2, R35.1, U24.3 (+): now also Q7.4 (Source)
- net at U18.5 (GATE): now also Q5.3 (Gate)
- net at R24.2, R26.1, U19.3 (+): now also Q5.4 (Source)
- net at U17.5 (GATE): now also Q4.3 (Gate)
- net at R23.1, R25.2, U16.3 (+): now also Q4.4 (Source)
- new net: C22.1, F1.2, Q4.1 (Drain), Q4.2 (Drain), Q4.5 (Drain), Q4.6 (Drain), U17.6 (SENSE), U17.8 (V+)
Other:
- moved on the sheet: D10, D11, D12, D13, D6, R14, R16, R23, R24, R25, R26, R31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
